Commit message: Make small tweaks + fixes

File: glennobi_description/urdf/glennobi.urdf.xacro (robot description, xacro)
@@ -22,7 +22,7 @@
 		<link name="${prefix}_wheel_link">
 			<visual>
-				<origin xyz="0 -0.045 0" rpy="${pi/2} 0 0"/>
+				<origin xyz="0 0 0" rpy="${pi/2} 0 0"/>
 				<geometry>
-					<mesh filename="package://glennobi_description/meshes/wheel.dae"/>
+					<cylinder radius="${wheelradius}" length="${wheelwidth}"/>
 				</geometry>
 			</visual>

Commit message: Updated all vals but bodyx and bodyz

File: glennobi_description/urdf/glennobi.urdf.xacro (robot description, xacro)
@@ -19,9 +19,8 @@
     <!-- Data from cad model
     X = -2.54667
-	Y = 0.68615
+	Y = .68615
 	Z = 9.90497
     Note not currently used but leaving here because might be useful later-->
-    <xacro:property name="bodyx" value="0"/>
-    <xacro:property name="bodyy" value="0"/>
+    <xacro:property name="bodyx" value="0.51"/>
     <xacro:property name="bodyz" value="-0.05"/>
     <!-- Controls tilt of robot model-->

Commit message: Updated all vals but bodyx and bodyz

File: glennobi_description/urdf/glennobi.urdf.xacro (robot description, xacro)
@@ -3,12 +3,23 @@
     <xacro:include filename="$(find glennobi_description)/urdf/glennobi.gazebo.xacro"/>
     <xacro:include filename="$(find glennobi_description)/urdf/glennobi.transmission.xacro"/>
-    <xacro:property name="bodylength" value="1.3"/>
-    <xacro:property name="bodywidth" value="0.43"/>
-    <xacro:property name="bodyheight" value="0.35"/>
-    <xacro:property name="wheelradius" value="0.232"/>
-    <xacro:property name="wheelwidth" value="0.12"/>
-    <xacro:property name="wheelsepx" value="0.28"/>
-    <xacro:property name="wheelsepy" value="0.4"/>
-    <xacro:property name="wheeloffsetx" value="0.13"/>
+    <!-- Units in Meters-->
+    <xacro:property name="bodylength" value="0.9411"/>
+    <xacro:property name="bodywidth" value="0.4577"/>
+    <xacro:property name="bodyheight" value="0.477"/>
+    <xacro:property name="wheelradius" value="0.1642"/>
+    <xacro:property name="wheelwidth" value="0.0635"/>
+    <!-- Distance from the centers of the wheels in the length and width of robot. -->
+    <!-- wheelsepx crosses through the robot -->
+    <xacro:property name="wheelsepx" value="0.3874"/>
+    <!-- wheelsepy is from wheel to wheel not crossing the center line-->
+    <xacro:property name="wheelsepy" value="0.386"/>
+    <!-- If wheels are not aligned use offset-->
+    <xacro:property name="wheeloffsetx" value="0.0"/>
+    <!-- body is for aligning the robot mesh to the center of gravity-->
+    <!-- Data from cad model
+    X = -2.54667
+	Y = .68615
+	Z = 9.90497
+    Note not currently used but leaving here because might be useful later-->
     <xacro:property name="bodyx" value="0.51"/>
     <xacro:property name="bodyz" value="-0.05"/>

Commit message: Model close to lining up

File: glennobi_description/urdf/glennobi.urdf.xacro (robot description, xacro)
@@ -19,8 +19,9 @@
     <!-- Data from cad model
     X = -2.54667
-	Y = .68615
+	Y = 0.68615
 	Z = 9.90497
     Note not currently used but leaving here because might be useful later-->
-    <xacro:property name="bodyx" value="0.51"/>
+    <xacro:property name="bodyx" value="0"/>
+    <xacro:property name="bodyy" value="0"/>
     <xacro:property name="bodyz" value="-0.05"/>
     <!-- Controls tilt of robot model-->

Commit message: Model close to lining up

File: glennobi_description/urdf/glennobi.urdf.xacro (robot description, xacro)
@@ -19,8 +19,9 @@
     <!-- Data from cad model
     X = -2.54667
-	Y = .68615
+	Y = 0.68615
 	Z = 9.90497
     Note not currently used but leaving here because might be useful later-->
-    <xacro:property name="bodyx" value="0.51"/>
+    <xacro:property name="bodyx" value="0"/>
+    <xacro:property name="bodyy" value="0"/>
     <xacro:property name="bodyz" value="-0.05"/>
     <xacro:macro name="default_inertial" params="mass">
@@ -64,5 +65,5 @@
     <link name="base_link">
         <visual>
-            <origin xyz="${bodyx} 0 ${bodyz}" rpy="${pi/2} 0 ${pi/2}"/>
+            <origin xyz="${bodyx} ${bodyy} ${bodyz}" rpy="0 0 ${pi/2}"/>
             <geometry>
                     <mesh filename="package://glennobi_description/meshes/chassis.dae"/>

Commit message: Model close to lining up

File: glennobi_description/urdf/glennobi.urdf.xacro (robot description, xacro)
@@ -3,13 +3,25 @@
     <xacro:include filename="$(find glennobi_description)/urdf/glennobi.gazebo.xacro"/>
     <xacro:include filename="$(find glennobi_description)/urdf/glennobi.transmission.xacro"/>
-    <xacro:property name="bodylength" value="1.3"/>
-    <xacro:property name="bodywidth" value="0.43"/>
-    <xacro:property name="bodyheight" value="0.35"/>
-    <xacro:property name="wheelradius" value="0.232"/>
-    <xacro:property name="wheelwidth" value="0.12"/>
-    <xacro:property name="wheelsepx" value="0.28"/>
-    <xacro:property name="wheelsepy" value="0.4"/>
-    <xacro:property name="wheeloffsetx" value="0.13"/>
-    <xacro:property name="bodyx" value="0.51"/>
+    <!-- Units in Meters-->
+    <xacro:property name="bodylength" value="0.9411"/>
+    <xacro:property name="bodywidth" value="0.4577"/>
+    <xacro:property name="bodyheight" value="0.477"/>
+    <xacro:property name="wheelradius" value="0.1642"/>
+    <xacro:property name="wheelwidth" value="0.0635"/>
+    <!-- Distance from the centers of the wheels in the length and width of robot. -->
+    <!-- wheelsepx crosses through the robot -->
+    <xacro:property name="wheelsepx" value="0.3874"/>
+    <!-- wheelsepy is from wheel to wheel not crossing the center line-->
+    <xacro:property name="wheelsepy" value="0.386"/>
+    <!-- If wheels are not aligned use offset-->
+    <xacro:property name="wheeloffsetx" value="0.0"/>
+    <!-- body is for aligning the robot mesh to the center of gravity-->
+    <!-- Data from cad model
+    X = -2.54667
+	Y = 0.68615
+	Z = 9.90497
+    Note not currently used but leaving here because might be useful later-->
+    <xacro:property name="bodyx" value="0"/>
+    <xacro:property name="bodyy" value="0"/>
     <xacro:property name="bodyz" value="-0.05"/>
     <xacro:macro name="default_inertial" params="mass">
@@ -53,5 +65,5 @@
     <link name="base_link">
         <visual>
-            <origin xyz="${bodyx} 0 ${bodyz}" rpy="${pi/2} 0 ${pi/2}"/>
+            <origin xyz="${bodyx} ${bodyy} ${bodyz}" rpy="0 0 ${pi/2}"/>
             <geometry>
                     <mesh filename="package://glennobi_description/meshes/chassis.dae"/>

Commit message: Added pitch yaw and roll to mesh variables

File: glennobi_description/urdf/glennobi.urdf.xacro (robot description, xacro)
@@ -45,4 +45,9 @@
     <xacro:property name="realpitch" value="${bodypitch}"/>
     <xacro:property name="realyaw" value="${bodyyaw}"/>
+    <!-- Controls tilt of robot model-->
+    <!-- Not yet sure if use pitch, yaw and roll to represent the correct rotations-->
+    <xacro:property name="bodypitch" value="0"/>
+    <xacro:property name="bodyyaw" value="0"/>
+    <xacro:property name="bodyroll" value="${pi/2}"/>
     <xacro:macro name="default_inertial" params="mass">
         <inertial>
@@ -85,5 +90,5 @@
     <link name="base_link">
         <visual>
-            <origin xyz="${bodyx} ${bodyy} ${bodyz}" rpy="${bodyroll} ${bodypitch} ${bodyyaw}"/>
+            <origin xyz="${bodyx} ${bodyy} ${bodyz}" rpy="${bodypitch} ${bodyyaw} ${bodyroll}"/>
             <geometry>
                     <mesh filename="package://glennobi_description/meshes/chassis.dae"/>

Commit message: Added pitch yaw and roll to mesh variables

File: glennobi_description/urdf/glennobi.urdf.xacro (robot description, xacro)
@@ -25,4 +25,9 @@
     <xacro:property name="bodyy" value="0"/>
     <xacro:property name="bodyz" value="-0.05"/>
+    <!-- Controls tilt of robot model-->
+    <!-- Not yet sure if use pitch, yaw and roll to represent the correct rotations-->
+    <xacro:property name="bodypitch" value="0"/>
+    <xacro:property name="bodyyaw" value="0"/>
+    <xacro:property name="bodyroll" value="${pi/2}"/>
     <xacro:macro name="default_inertial" params="mass">
         <inertial>
@@ -65,5 +70,5 @@
     <link name="base_link">
         <visual>
-            <origin xyz="${bodyx} ${bodyy} ${bodyz}" rpy="0 0 ${pi/2}"/>
+            <origin xyz="${bodyx} ${bodyy} ${bodyz}" rpy="${bodypitch} ${bodyyaw} ${bodyroll}"/>
             <geometry>
                     <mesh filename="package://glennobi_description/meshes/chassis.dae"/>

Commit message: Finshed updating all values I know about

File: glennobi_description/urdf/glennobi.urdf.xacro (robot description, xacro)
@@ -50,4 +50,19 @@
     <xacro:property name="bodyyaw" value="0"/>
     <xacro:property name="bodyroll" value="${pi/2}"/>
+    <!-- Note line up robot model first or you will spend time realigning the other sensors-->
+    <!-- Values for RealSense-->
+    <!-- Values for overall dimensions of RealSense-->
+    <xacro:property name="reallength" value="0.0758"/>
+    <xacro:property name="realwidth" value="0.025"/>
+    <xacro:property name="realheight" value="0.0151"/>
+    <!-- Values from center of Body to the RealSense-->
+    <xacro:property name="realx" value="${0.35+bodyx}"/>
+    <xacro:property name="realy" value="${0.145+bodyy}"/>
+    <xacro:property name="realz" value="${-0.01+bodyz}"/>
+    <!-- Controls tilt of RealSense model-->
+    <!-- Not yet sure if use pitch, yaw and roll to represent the correct rotations-->
+    <xacro:property name="realpitch" value="${bodypitch + (20.42)*pi/180}"/>
+    <xacro:property name="realyaw" value="${bodyyaw}"/>
+    <xacro:property name="realroll" value="${bodyroll}"/>
     <xacro:macro name="default_inertial" params="mass">
         <inertial>

Commit message: Finshed updating all values I know about

File: glennobi_description/urdf/glennobi.urdf.xacro (robot description, xacro)
@@ -3,15 +3,17 @@
     <xacro:include filename="$(find glennobi_description)/urdf/glennobi.gazebo.xacro"/>
     <xacro:include filename="$(find glennobi_description)/urdf/glennobi.transmission.xacro"/>
+    <!-- NOTE Length=x, Width=y, Height=z-->
+    <!-- Values for the robot body-->
     <!-- Units in Meters-->
     <xacro:property name="bodylength" value="0.9411"/>
     <xacro:property name="bodywidth" value="0.4577"/>
     <xacro:property name="bodyheight" value="0.477"/>
-    <xacro:property name="wheelradius" value="0.1642"/>
-    <xacro:property name="wheelwidth" value="0.0635"/>
+    <xacro:property name="wheelradius" value="0.1561"/>
+    <xacro:property name="wheelwidth" value="0.0762"/>
     <!-- Distance from the centers of the wheels in the length and width of robot. -->
-    <!-- wheelsepx crosses through the robot -->
-    <xacro:property name="wheelsepx" value="0.3874"/>
+    <!-- wheelsepx distance from spoke to spoke over 2 -->
+    <xacro:property name="wheelsepx" value="${0.3947/2}"/>
     <!-- wheelsepy is from wheel to wheel not crossing the center line-->
-    <xacro:property name="wheelsepy" value="0.386"/>
+    <xacro:property name="wheelsepy" value="0.3175"/>
     <!-- If wheels are not aligned use offset-->
     <xacro:property name="wheeloffsetx" value="0.0"/>
@@ -22,7 +24,7 @@
 	Z = 9.90497
     Note not currently used but leaving here because might be useful later-->
-    <xacro:property name="bodyx" value="0"/>
-    <xacro:property name="bodyy" value="0"/>
-    <xacro:property name="bodyz" value="-0.05"/>
+    <xacro:property name="bodyx" value="0.13"/>
+    <xacro:property name="bodyy" value="0.01"/>
+    <xacro:property name="bodyz" value="0.12"/>
     <!-- Controls tilt of robot model-->
     <!-- Not yet sure if use pitch, yaw and roll to represent the correct rotations-->
@@ -30,4 +32,19 @@
     <xacro:property name="bodyyaw" value="0"/>
     <xacro:property name="bodyroll" value="${pi/2}"/>
+    <!-- Note line up robot model first or you will spend time realigning the other sensors-->
+    <!-- Values for RealSense-->
+    <!-- Values for overall dimensions of RealSense-->
+    <xacro:property name="reallength" value="0.0758"/>
+    <xacro:property name="realwidth" value="0.025"/>
+    <xacro:property name="realheight" value="0.0151"/>
+    <!-- Values from center of Body to the RealSense-->
+    <xacro:property name="realx" value="${0.35+bodyx}"/>
+    <xacro:property name="realy" value="${0.145+bodyy}"/>
+    <xacro:property name="realz" value="${-0.01+bodyz}"/>
+    <!-- Controls tilt of RealSense model-->
+    <!-- Not yet sure if use pitch, yaw and roll to represent the correct rotations-->
+    <xacro:property name="realpitch" value="${bodypitch + (20.42)*pi/180}"/>
+    <xacro:property name="realyaw" value="${bodyyaw}"/>
+    <xacro:property name="realroll" value="${bodyroll}"/>
     <xacro:macro name="default_inertial" params="mass">
         <inertial>
@@ -76,5 +93,5 @@
         </visual>
         <collision>
-            <origin xyz="${bodyx} 0 ${bodyz}" rpy="${pi/2} 0 ${pi/2}"/>
+            <origin xyz="${bodyx} ${bodyy} ${bodyz}" rpy="${bodypitch} ${bodyyaw} ${bodyroll}"/>
             <geometry>
                 <mesh filename="package://glennobi_description/meshes/chassis.dae"/>
@@ -94,5 +111,5 @@
         <visual>
             <geometry>
-                <box size="0.1 0.025 0.015"/>
+                <box size="${reallength} ${realwidth} ${realheight}"/>
             </geometry>
         </visual>
@@ -102,6 +119,7 @@
         <child link="realsense_link"/>
         <!-- transform from base_link with additional 20 degree tilt down -->
-        <origin xyz="-0.57 0 0.33" rpy="${-(20+90)*pi/180} 0 ${pi/2}"/>
+        <origin xyz="${realx} ${realy} ${realz}" rpy="${realpitch} ${realyaw} ${realroll}"/>
     </joint>
+    <!-- Waiting on this location from CAD people-->
     <link name="imu_link"/>
     <joint name="imu_joint" type="fixed">

Commit message: Updated all values

File: glennobi_description/urdf/glennobi.urdf.xacro (robot description, xacro)
@@ -58,5 +58,5 @@
     <!-- Values from center of Body to the RealSense-->
     <xacro:property name="realx" value="${0.35+bodyx}"/>
-    <xacro:property name="realy" value="${0.145+bodyy}"/>
+    <xacro:property name="realy" value="${0.152+bodyy}"/>
     <xacro:property name="realz" value="${-0.01+bodyz}"/>
     <!-- Controls tilt of RealSense model-->

Commit message: Updated all values

File: glennobi_description/urdf/glennobi.urdf.xacro (robot description, xacro)
@@ -40,5 +40,5 @@
     <!-- Values from center of Body to the RealSense-->
     <xacro:property name="realx" value="${0.35+bodyx}"/>
-    <xacro:property name="realy" value="${0.145+bodyy}"/>
+    <xacro:property name="realy" value="${0.152+bodyy}"/>
     <xacro:property name="realz" value="${-0.01+bodyz}"/>
     <!-- Controls tilt of RealSense model-->

Commit message: Fixed errors in pitch yaw and roll

File: glennobi_description/urdf/glennobi.urdf.xacro (robot description, xacro)
@@ -28,8 +28,7 @@
     <xacro:property name="bodyz" value="0.12"/>
     <!-- Controls tilt of robot model-->
-    <!-- Not yet sure if use pitch, yaw and roll to represent the correct rotations-->
+    <xacro:property name="bodyroll" value="0"/>
     <xacro:property name="bodypitch" value="0"/>
-    <xacro:property name="bodyyaw" value="0"/>
-    <xacro:property name="bodyroll" value="${pi/2}"/>
+    <xacro:property name="bodyyaw" value="${pi/2}"/>
     <!-- Note line up robot model first or you will spend time realigning the other sensors-->
     <!-- Values for RealSense-->
@@ -43,8 +42,7 @@
     <xacro:property name="realz" value="${-0.01+bodyz}"/>
     <!-- Controls tilt of RealSense model-->
-    <!-- Not yet sure if use pitch, yaw and roll to represent the correct rotations-->
-    <xacro:property name="realpitch" value="${bodypitch + (20.42)*pi/180}"/>
-    <xacro:property name="realyaw" value="${bodyyaw}"/>
-    <xacro:property name="realroll" value="${bodyroll}"/>
+    <xacro:property name="realroll" value="${bodypitch + (20.42)*pi/180}"/>
+    <xacro:property name="realpitch" value="${bodyyaw}"/>
+    <xacro:property name="realyaw" value="${bodyroll}"/>
     <xacro:macro name="default_inertial" params="mass">
         <inertial>

Commit message: Fixed errors in pitch yaw and roll

File: glennobi_description/urdf/glennobi.urdf.xacro (robot description, xacro)
@@ -48,6 +48,5 @@
     <!-- Not yet sure if use pitch, yaw and roll to represent the correct rotations-->
     <xacro:property name="bodypitch" value="0"/>
-    <xacro:property name="bodyyaw" value="0"/>
-    <xacro:property name="bodyroll" value="${pi/2}"/>
+    <xacro:property name="bodyyaw" value="${pi/2}"/>
     <!-- Note line up robot model first or you will spend time realigning the other sensors-->
     <!-- Values for RealSense-->
@@ -61,8 +60,7 @@
     <xacro:property name="realz" value="${-0.01+bodyz}"/>
     <!-- Controls tilt of RealSense model-->
-    <!-- Not yet sure if use pitch, yaw and roll to represent the correct rotations-->
-    <xacro:property name="realpitch" value="${bodypitch + (20.42)*pi/180}"/>
-    <xacro:property name="realyaw" value="${bodyyaw}"/>
-    <xacro:property name="realroll" value="${bodyroll}"/>
+    <xacro:property name="realroll" value="${bodypitch + (20.42)*pi/180}"/>
+    <xacro:property name="realpitch" value="${bodyyaw}"/>
+    <xacro:property name="realyaw" value="${bodyroll}"/>
     <xacro:macro name="default_inertial" params="mass">
         <inertial>

Commit message: Fixed bug where variables were not updated

File: glennobi_description/urdf/glennobi.urdf.xacro (robot description, xacro)
@@ -45,22 +45,4 @@
     <xacro:property name="realpitch" value="${bodypitch}"/>
     <xacro:property name="realyaw" value="${bodyyaw}"/>
-    <!-- Controls tilt of robot model-->
-    <!-- Not yet sure if use pitch, yaw and roll to represent the correct rotations-->
-    <xacro:property name="bodypitch" value="0"/>
-    <xacro:property name="bodyyaw" value="${pi/2}"/>
-    <!-- Note line up robot model first or you will spend time realigning the other sensors-->
-    <!-- Values for RealSense-->
-    <!-- Values for overall dimensions of RealSense-->
-    <xacro:property name="reallength" value="0.0758"/>
-    <xacro:property name="realwidth" value="0.025"/>
-    <xacro:property name="realheight" value="0.0151"/>
-    <!-- Values from center of Body to the RealSense-->
-    <xacro:property name="realx" value="${0.35+bodyx}"/>
-    <xacro:property name="realy" value="${0.152+bodyy}"/>
-    <xacro:property name="realz" value="${-0.01+bodyz}"/>
-    <!-- Controls tilt of RealSense model-->
-    <xacro:property name="realroll" value="${bodypitch + (20.42)*pi/180}"/>
-    <xacro:property name="realpitch" value="${bodyyaw}"/>
-    <xacro:property name="realyaw" value="${bodyroll}"/>
     <xacro:macro name="default_inertial" params="mass">
         <inertial>
@@ -103,5 +85,5 @@
     <link name="base_link">
         <visual>
-            <origin xyz="${bodyx} ${bodyy} ${bodyz}" rpy="${bodypitch} ${bodyyaw} ${bodyroll}"/>
+            <origin xyz="${bodyx} ${bodyy} ${bodyz}" rpy="${bodyroll} ${bodypitch} ${bodyyaw}"/>
             <geometry>
                     <mesh filename="package://glennobi_description/meshes/chassis.dae"/>

Commit message: Fixed bug where variables were not updated

File: glennobi_description/urdf/glennobi.urdf.xacro (robot description, xacro)
@@ -42,7 +42,7 @@
     <xacro:property name="realz" value="${-0.01+bodyz}"/>
     <!-- Controls tilt of RealSense model-->
-    <xacro:property name="realroll" value="${bodypitch + (20.42)*pi/180}"/>
-    <xacro:property name="realpitch" value="${bodyyaw}"/>
-    <xacro:property name="realyaw" value="${bodyroll}"/>
+    <xacro:property name="realroll" value="${bodyroll + (20.42)*pi/180}"/>
+    <xacro:property name="realpitch" value="${bodypitch}"/>
+    <xacro:property name="realyaw" value="${bodyyaw}"/>
     <xacro:macro name="default_inertial" params="mass">
         <inertial>
@@ -85,5 +85,5 @@
     <link name="base_link">
         <visual>
-            <origin xyz="${bodyx} ${bodyy} ${bodyz}" rpy="${bodypitch} ${bodyyaw} ${bodyroll}"/>
+            <origin xyz="${bodyx} ${bodyy} ${bodyz}" rpy="${bodyroll} ${bodypitch} ${bodyyaw}"/>
             <geometry>
                     <mesh filename="package://glennobi_description/meshes/chassis.dae"/>
@@ -91,5 +91,5 @@
         </visual>
         <collision>
-            <origin xyz="${bodyx} ${bodyy} ${bodyz}" rpy="${bodypitch} ${bodyyaw} ${bodyroll}"/>
+            <origin xyz="${bodyx} ${bodyy} ${bodyz}" rpy="${bodyroll} ${bodypitch} ${bodyyaw}"/>
             <geometry>
                 <mesh filename="package://glennobi_description/meshes/chassis.dae"/>
@@ -117,5 +117,5 @@
         <child link="realsense_link"/>
         <!-- transform from base_link with additional 20 degree tilt down -->
-        <origin xyz="${realx} ${realy} ${realz}" rpy="${realpitch} ${realyaw} ${realroll}"/>
+        <origin xyz="${realx} ${realy} ${realz}" rpy="${realroll} ${realpitch} ${realyaw}"/>
     </joint>
     <!-- Waiting on this location from CAD people-->
