Commit message: Hopefully Squashed properly

File: glennobi_description/urdf/glennobi.urdf.xacro (robot description, xacro)
@@ -3,14 +3,46 @@
     <xacro:include filename="$(find glennobi_description)/urdf/glennobi.gazebo.xacro"/>
     <xacro:include filename="$(find glennobi_description)/urdf/glennobi.transmission.xacro"/>
-    <xacro:property name="bodylength" value="1.3"/>
-    <xacro:property name="bodywidth" value="0.43"/>
-    <xacro:property name="bodyheight" value="0.35"/>
-    <xacro:property name="wheelradius" value="0.232"/>
-    <xacro:property name="wheelwidth" value="0.12"/>
-    <xacro:property name="wheelsepx" value="0.28"/>
-    <xacro:property name="wheelsepy" value="0.4"/>
-    <xacro:property name="wheeloffsetx" value="0.13"/>
-    <xacro:property name="bodyx" value="0.51"/>
-    <xacro:property name="bodyz" value="-0.05"/>
+    <!-- NOTE Length=x, Width=y, Height=z-->
+    <!-- Values for the robot body-->
+    <!-- Units in Meters-->
+    <xacro:property name="bodylength" value="0.9411"/>
+    <xacro:property name="bodywidth" value="0.4577"/>
+    <xacro:property name="bodyheight" value="0.477"/>
+    <xacro:property name="wheelradius" value="0.1561"/>
+    <xacro:property name="wheelwidth" value="0.0762"/>
+    <!-- Distance from the centers of the wheels in the length and width of robot. -->
+    <!-- wheelsepx distance from spoke to spoke over 2 -->
+    <xacro:property name="wheelsepx" value="${0.3947/2}"/>
+    <!-- wheelsepy is from wheel to wheel not crossing the center line-->
+    <xacro:property name="wheelsepy" value="0.3175"/>
+    <!-- If wheels are not aligned use offset-->
+    <xacro:property name="wheeloffsetx" value="0.0"/>
+    <!-- body is for aligning the robot mesh to the center of gravity-->
+    <!-- Data from cad model
+    X = -2.54667
+	Y = 0.68615
+	Z = 9.90497
+    Note not currently used but leaving here because might be useful later-->
+    <xacro:property name="bodyx" value="0.13"/>
+    <xacro:property name="bodyy" value="0.01"/>
+    <xacro:property name="bodyz" value="0.12"/>
+    <!-- Controls tilt of robot model-->
+    <xacro:property name="bodyroll" value="0"/>
+    <xacro:property name="bodypitch" value="0"/>
+    <xacro:property name="bodyyaw" value="${pi/2}"/>
+    <!-- Note line up robot model first or you will spend time realigning the other sensors-->
+    <!-- Values for RealSense-->
+    <!-- Values for overall dimensions of RealSense-->
+    <xacro:property name="reallength" value="0.0758"/>
+    <xacro:property name="realwidth" value="0.025"/>
+    <xacro:property name="realheight" value="0.0151"/>
+    <!-- Values from center of Body to the RealSense-->
+    <xacro:property name="realx" value="${0.35+bodyx}"/>
+    <xacro:property name="realy" value="${0.152+bodyy}"/>
+    <xacro:property name="realz" value="${-0.01+bodyz}"/>
+    <!-- Controls tilt of RealSense model-->
+    <xacro:property name="realroll" value="${bodyroll + (20.42)*pi/180}"/>
+    <xacro:property name="realpitch" value="${bodypitch}"/>
+    <xacro:property name="realyaw" value="${bodyyaw}"/>
     <xacro:macro name="default_inertial" params="mass">
         <inertial>
@@ -53,5 +85,5 @@
     <link name="base_link">
         <visual>
-            <origin xyz="${bodyx} 0 ${bodyz}" rpy="${pi/2} 0 ${pi/2}"/>
+            <origin xyz="${bodyx} ${bodyy} ${bodyz}" rpy="${bodyroll} ${bodypitch} ${bodyyaw}"/>
             <geometry>
                     <mesh filename="package://glennobi_description/meshes/chassis.dae"/>
@@ -59,5 +91,5 @@
         </visual>
         <collision>
-            <origin xyz="${bodyx} 0 ${bodyz}" rpy="${pi/2} 0 ${pi/2}"/>
+            <origin xyz="${bodyx} ${bodyy} ${bodyz}" rpy="${bodyroll} ${bodypitch} ${bodyyaw}"/>
             <geometry>
                 <mesh filename="package://glennobi_description/meshes/chassis.dae"/>
@@ -77,5 +109,5 @@
         <visual>
             <geometry>
-                <box size="0.1 0.025 0.015"/>
+                <box size="${reallength} ${realwidth} ${realheight}"/>
             </geometry>
         </visual>
@@ -85,6 +117,7 @@
         <child link="realsense_link"/>
         <!-- transform from base_link with additional 20 degree tilt down -->
-        <origin xyz="-0.57 0 0.33" rpy="${-(20+90)*pi/180} 0 ${pi/2}"/>
+        <origin xyz="${realx} ${realy} ${realz}" rpy="${realroll} ${realpitch} ${realyaw}"/>
     </joint>
+    <!-- Waiting on this location from CAD people-->
     <link name="imu_link"/>
     <joint name="imu_joint" type="fixed">

Commit message: added inertia and fixed realsense

File: glennobi_description/urdf/glennobi.urdf.xacro (robot description, xacro)
@@ -42,7 +42,30 @@
     <xacro:property name="realz" value="${-0.01+bodyz}"/>
     <!-- Controls tilt of RealSense model-->
-    <xacro:property name="realroll" value="${bodyroll + (20.42)*pi/180}"/>
-    <xacro:property name="realpitch" value="${bodypitch}"/>
+    <xacro:property name="realroll" value="${bodyroll + (20.42+90)*pi/180}"/>
+    <xacro:property name="realpitch" value="${bodypitch +pi}"/>
     <xacro:property name="realyaw" value="${bodyyaw}"/>
+    <!-- Inertia Section-->
+    <!-- Cadders Inertia Offset-->
+    <xacro:property name="robotlengthfromzero" value="-0.282549"/>
+    <xacro:property name="robotwidthfromzero" value="0.85221"/>
+    <xacro:property name="robotheightfromzero" value="-9.8254"/>
+    <!-- Masses unit kg-->
+    <xacro:property name="wheelmass" value="1.05216"/>
+    <!-- Mass of robot without wheels-->
+    <xacro:property name="robotmass" value="30.8"/>
+    <!-- Inertial values for robot units kg/m^2-->
+    <xacro:property name="robotlxx" value="0.385"/>
+    <xacro:property name="robotlxy" value="0"/>
+    <xacro:property name="robotlxz" value="0"/>
+    <xacro:property name="robotlyy" value="1.92098166"/>
+    <xacro:property name="robotlyz" value="0"/>
+    <xacro:property name="robotlzz" value="1.844169"/>
+    <!-- Inertial values for wheels units kg/m^2-->
+    <xacro:property name="wheellxx" value="${1/12*wheelmass*(3*wheelradius*wheelradius+wheelwidth*wheelwidth)}"/>
+    <xacro:property name="wheellxy" value="0.0"/>
+    <xacro:property name="wheellxz" value="0"/>
+    <xacro:property name="wheellyy" value="${1/2*wheelmass*wheelradius*wheelradius}"/>
+    <xacro:property name="wheellyz" value="0.0"/>
+    <xacro:property name="wheellzz" value="${wheellxx}"/>
     <xacro:macro name="default_inertial" params="mass">
         <inertial>
@@ -67,6 +90,6 @@
             </collision>
             <inertial>
-                <mass value="1.6"/>
-                <inertia ixx="0.035" ixy="0.0" ixz="0.0" iyy="0.035" iyz="0.0" izz="0.06" />
+                <mass value="${wheelmass}"/>
+                <inertia ixx="${wheellxx}" ixy="${wheellxy}" ixz="${wheellxz}" iyy="${wheellyy}" iyz="${wheellyz}" izz="${wheellzz}" />
             </inertial>
         </link>
@@ -98,6 +121,6 @@
         </collision>
         <inertial>
-            <mass value="16"/>
-            <inertia ixx="4.5" ixy="0.0" ixz="0.0" iyy="4.5" iyz="0.0" izz="0.8" />
+            <mass value="${robotmass}"/>
+            <inertia ixx="${robotlxx}" ixy="${robotlxy}" ixz="${robotlxz}" iyy="${robotlyy}" iyz="${robotlyz}" izz="${robotlzz}" />
         </inertial>
     </link>

Commit message: Updated variables.

File: glennobi_description/urdf/glennobi.urdf.xacro (robot description, xacro)
@@ -6,6 +6,6 @@
     <!-- Values for the robot body-->
     <!-- Units in Meters-->
-    <xacro:property name="bodylength" value="0.9411"/>
-    <xacro:property name="bodywidth" value="0.4577"/>
+    <xacro:property name="bodylength" value="0.4577"/>
+    <xacro:property name="bodywidth" value="0.9411"/>
     <xacro:property name="bodyheight" value="0.477"/>
     <xacro:property name="wheelradius" value="0.1561"/>
@@ -42,6 +42,6 @@
     <xacro:property name="realz" value="${-0.01+bodyz}"/>
     <!-- Controls tilt of RealSense model-->
-    <xacro:property name="realroll" value="${bodyroll + (20.42+90)*pi/180}"/>
-    <xacro:property name="realpitch" value="${bodypitch +pi}"/>
+    <xacro:property name="realroll" value="${(20.42+90)*pi/180}"/>
+    <xacro:property name="realpitch" value="${bodypitch+pi}"/>
     <xacro:property name="realyaw" value="${bodyyaw}"/>
     <!-- Inertia Section-->
@@ -116,6 +116,6 @@
             <origin xyz="${bodyx} ${bodyy} ${bodyz}" rpy="${bodyroll} ${bodypitch} ${bodyyaw}"/>
             <geometry>
-                <mesh filename="package://glennobi_description/meshes/chassis.dae"/>
-                <!-- box size="${bodylength} ${bodywidth} ${bodyheight}"/-->
+                <!-- <mesh filename="package://glennobi_description/meshes/chassis.dae"/> -->
+                <box size="${bodylength} ${bodywidth} ${bodyheight}"/>
             </geometry>
         </collision>

Commit message: Made camera more accurate.

File: glennobi_description/urdf/glennobi.urdf.xacro (robot description, xacro)
@@ -42,5 +42,5 @@
     <xacro:property name="realz" value="${-0.01+bodyz}"/>
     <!-- Controls tilt of RealSense model-->
-    <xacro:property name="realroll" value="${(20.42+90)*pi/180}"/>
+    <xacro:property name="realroll" value="${(0+90)*pi/180}"/>
     <xacro:property name="realpitch" value="${bodypitch+pi}"/>
     <xacro:property name="realyaw" value="${bodyyaw}"/>

Commit message: Fixed camera angle.

File: glennobi_description/urdf/glennobi.urdf.xacro (robot description, xacro)
@@ -42,6 +42,6 @@
     <xacro:property name="realz" value="${-0.01+bodyz}"/>
     <!-- Controls tilt of RealSense model-->
-    <xacro:property name="realroll" value="${(0+90)*pi/180}"/>
-    <xacro:property name="realpitch" value="${bodypitch+pi}"/>
+    <xacro:property name="realroll" value="${bodyroll + (20.42+90)*pi/180}"/>
+    <xacro:property name="realpitch" value="${bodypitch}"/>
     <xacro:property name="realyaw" value="${bodyyaw}"/>
     <!-- Inertia Section-->

Commit message: Fix a few camera transforms

File: glennobi_description/urdf/glennobi.urdf.xacro (robot description, xacro)
@@ -42,7 +42,7 @@
     <xacro:property name="realz" value="${-0.01+bodyz}"/>
     <!-- Controls tilt of RealSense model-->
-    <xacro:property name="realroll" value="${bodyroll + (20.42+90)*pi/180}"/>
-    <xacro:property name="realpitch" value="${bodypitch}"/>
-    <xacro:property name="realyaw" value="${bodyyaw}"/>
+    <xacro:property name="realroll" value="${-(20.42 + 90) * pi/180}"/>
+    <xacro:property name="realpitch" value="0"/>
+    <xacro:property name="realyaw" value="${-pi/2}"/>
     <!-- Inertia Section-->
     <!-- Cadders Inertia Offset-->
@@ -116,6 +116,6 @@
             <origin xyz="${bodyx} ${bodyy} ${bodyz}" rpy="${bodyroll} ${bodypitch} ${bodyyaw}"/>
             <geometry>
-                <!-- <mesh filename="package://glennobi_description/meshes/chassis.dae"/> -->
-                <box size="${bodylength} ${bodywidth} ${bodyheight}"/>
+                <mesh filename="package://glennobi_description/meshes/chassis.dae"/>
+                <!-- <box size="${bodylength} ${bodywidth} ${bodyheight}"/> -->
             </geometry>
         </collision>

Commit message: Add inertia of cylinder macro

File: glennobi_description/urdf/glennobi.urdf.xacro (robot description, xacro)
@@ -62,10 +62,9 @@
     <xacro:property name="robotlzz" value="1.844169"/>
     <!-- Inertial values for wheels units kg/m^2-->
-    <xacro:property name="wheellxx" value="${1/12*wheelmass*(3*wheelradius*wheelradius+wheelwidth*wheelwidth)}"/>
-    <xacro:property name="wheellxy" value="0.0"/>
-    <xacro:property name="wheellxz" value="0.0"/>
-    <xacro:property name="wheellyy" value="${1/2*wheelmass*wheelradius*wheelradius}"/>
-    <xacro:property name="wheellyz" value="0.0"/>
-    <xacro:property name="wheellzz" value="${wheellxx}"/>
+    <xacro:macro name="cylinder_inertia" params="m r h">
+      <inertia  ixx="${m*(3*r*r+h*h)/12}" ixy = "0" ixz = "0"
+        iyy="${m*(3*r*r+h*h)/12}" iyz = "0"
+        izz="${m*r*r/2}"/>
+    </xacro:macro>
     <xacro:macro name="wheel" params="prefix side reflect">
         <link name="${prefix}_wheel_link">
@@ -84,6 +83,7 @@
             </collision>
             <inertial>
+                <origin xyz="0 0 0" rpy="${pi/2} 0 0" />
                 <mass value="${wheelmass}"/>
-                <inertia ixx="${wheellxx}" ixy="${wheellxy}" ixz="${wheellxz}" iyy="${wheellyy}" iyz="${wheellyz}" izz="${wheellzz}" />
+                <xacro:cylinder_inertia m="${wheelmass}" r="${wheelradius}" h="${wheelwidth}"/>
             </inertial>
         </link>
