Commit message: Make tweaks to get gazebo path following simulation working

File: glennobi_description/urdf/glennobi.gazebo.xacro (robot description, xacro)
@@ -13,5 +13,5 @@
 	<gazebo reference="realsense_link">
 		<sensor name="realsense_camera" type="depth">
-			<update_rate>20</update_rate>
+			<update_rate>10</update_rate>
 			<camera>
 				<horizontal_fov>1.047198</horizontal_fov>
@@ -22,6 +22,6 @@
 				</image>
 				<clip>
-					<near>0.05</near>
-					<far>4</far>
+					<near>0.2</near>
+					<far>4.0</far>
 				</clip>
 			</camera>
@@ -36,5 +36,5 @@
 				<depthImageInfoTopicName>depth/camera_info</depthImageInfoTopicName>
 				<pointCloudTopicName>depth/points</pointCloudTopicName>
-				<pointCloudCutoff>0.5</pointCloudCutoff>
+				<pointCloudCutoff>0.2</pointCloudCutoff>
 				<pointCloudCutoffMax>4.0</pointCloudCutoffMax>
 				<distortionK1>0.0</distortionK1>
@@ -50,4 +50,17 @@
 		</sensor>
 	</gazebo>
+	<!-- gazebo_ros_p3d for position groundtruth -->
+	<gazebo>
+		<plugin name="p3d_base_link_controller" filename="libcustom_p3d_plugin.so">
+				<alwaysOn>true</alwaysOn>
+				<updateRate>5.0</updateRate>
+				<bodyName>base_link</bodyName>
+				<topicName>/uwb_nodes</topicName>
+				<frameName>map</frameName>
+				<xyzOffsets>0 0 0</xyzOffsets>
+				<rpyOffsets>0 0 0</rpyOffsets>
+				<gaussianNoise>0.15</gaussianNoise>
+		</plugin>
+	</gazebo>
   <!-- Gazebo plugin for ROS Control -->
   <gazebo>

File: glennobi_description/urdf/glennobi.urdf.xacro (robot description, xacro)
@@ -84,5 +84,5 @@
 		<parent link="base_link"/>
 		<child link="realsense_link"/>
-		<origin xyz="-0.57 0 0.21" rpy="0 ${10*pi/180} ${pi}"/>
+		<origin xyz="-0.57 0 0.33" rpy="0 ${20*pi/180} ${pi}"/>
 	</joint>
 </robot>

Commit message: Add imu to realsense and simplify its depth frame

File: glennobi_description/urdf/glennobi.gazebo.xacro (robot description, xacro)
@@ -15,4 +15,5 @@
 			<update_rate>10</update_rate>
 			<camera>
+				<pose>0 0 0 ${pi/2} ${-pi/2} 0</pose>
 				<horizontal_fov>1.5708</horizontal_fov>
 				<image>
@@ -30,5 +31,5 @@
 				<updateRate>0.0</updateRate>
 				<cameraName>realsense</cameraName>
-				<frameName>realsense_depth_link</frameName>
+				<frameName>realsense_link</frameName>
 				<imageTopicName>color/image_raw</imageTopicName>
 				<cameraInfoTopicName>color/camera_info</cameraInfoTopicName>
@@ -63,7 +64,26 @@
 		</plugin>
 	</gazebo>
+	<gazebo reference="realsense_link">
+    <gravity>true</gravity>
+    <sensor name="imu_realsense" type="imu">
+      <always_on>true</always_on>
+      <update_rate>20</update_rate>
+      <visualize>false</visualize>
+      <plugin name="imu_plugin" filename="libgazebo_ros_imu_sensor.so">
+        <topicName>imu_realsense/data_raw</topicName>
+        <bodyName>realsense_link</bodyName>
+        <updateRateHZ>100.0</updateRateHZ>
+        <gaussianNoise>0.0</gaussianNoise>
+        <xyzOffset>0 0 0</xyzOffset>
+        <rpyOffset>${-20*pi/180} 0 0</rpyOffset>
+        <frameName>realsense_link</frameName>
+        <initialOrientationAsReference>false</initialOrientationAsReference>
+      </plugin>
+    </sensor>
+  </gazebo>
   <!-- Gazebo plugin for ROS Control -->
   <gazebo>
     <plugin name="gazebo_ros_control" filename="libgazebo_ros_control.so">
+			<legacyModeNS>true</legacyModeNS>
       <robotNamespace>/</robotNamespace>
     </plugin>

File: glennobi_description/urdf/glennobi.urdf.xacro (robot description, xacro)
@@ -77,5 +77,5 @@
 		<visual>
 			<geometry>
-				<box size="0.015 0.1 0.025"/>
+				<box size="0.1 0.025 0.015"/>
 			</geometry>
 		</visual>
@@ -84,5 +84,6 @@
 		<parent link="base_link"/>
 		<child link="realsense_link"/>
-		<origin xyz="-0.57 0 0.33" rpy="0 ${20*pi/180} ${pi}"/>
+		<!-- transform from base_link with additional 20 degree tilt down -->
+		<origin xyz="-0.57 0 0.33" rpy="${-(20+90)*pi/180} 0 ${pi/2}"/>
 	</joint>
 </robot>

Commit message: Adjust a few kalman filter and sensor things

File: glennobi_description/urdf/glennobi.gazebo.xacro (robot description, xacro)
@@ -1,89 +1,109 @@
 <?xml version="1.0"?>
 <robot name="glennobi_gazebo_description" xmlns:xacro="http://www.ros.org/wiki/xacro">
-	<xacro:macro name="wheel_gazebo" params="prefix">
-		<gazebo reference="${prefix}_wheel_link">
-			<material>Gazebo/Grey</material>
-			<mu1>3</mu1>
-			<mu2>3</mu2>
-		</gazebo>
-	</xacro:macro>
-	<gazebo reference="base_link">
-		<material>Gazebo/Blue</material>
-	</gazebo>
-	<gazebo reference="realsense_link">
-		<sensor name="realsense_camera" type="depth">
-			<update_rate>10</update_rate>
-			<camera>
-				<pose>0 0 0 ${pi/2} ${-pi/2} 0</pose>
-				<horizontal_fov>1.5708</horizontal_fov>
-				<image>
-					<width>640</width>
-					<height>480</height>
-					<format>R8G8B8</format>
-				</image>
-				<clip>
-					<near>0.2</near>
-					<far>4.0</far>
-				</clip>
-			</camera>
-			<plugin name="depth_camera_plugin" filename="libgazebo_ros_openni_kinect.so">
-				<alwaysOn>true</alwaysOn>
-				<updateRate>0.0</updateRate>
-				<cameraName>realsense</cameraName>
-				<frameName>realsense_link</frameName>
-				<imageTopicName>color/image_raw</imageTopicName>
-				<cameraInfoTopicName>color/camera_info</cameraInfoTopicName>
-				<depthImageTopicName>depth/image_raw</depthImageTopicName>
-				<depthImageInfoTopicName>depth/camera_info</depthImageInfoTopicName>
-				<pointCloudTopicName>depth/points</pointCloudTopicName>
-				<pointCloudCutoff>0.2</pointCloudCutoff>
-				<pointCloudCutoffMax>4.0</pointCloudCutoffMax>
-				<distortionK1>0.0</distortionK1>
-				<distortionK2>0.0</distortionK2>
-				<distortionK3>0.0</distortionK3>
-				<distortionT1>0.0</distortionT1>
-				<distortionT2>0.0</distortionT2>
-				<CxPrime>0</CxPrime>
-				<Cx>0</Cx>
-				<Cy>0</Cy>
-				<focalLength>0</focalLength>
-			</plugin>
-		</sensor>
-	</gazebo>
-	<!-- gazebo_ros_p3d for position groundtruth -->
-	<gazebo>
-		<plugin name="p3d_base_link_controller" filename="libcustom_p3d_plugin.so">
-				<alwaysOn>true</alwaysOn>
-				<updateRate>5.0</updateRate>
-				<bodyName>base_link</bodyName>
-				<topicName>/uwb_nodes</topicName>
-				<frameName>map</frameName>
-				<xyzOffsets>0 0 0</xyzOffsets>
-				<rpyOffsets>0 0 0</rpyOffsets>
-				<gaussianNoise>0.15</gaussianNoise>
-		</plugin>
-	</gazebo>
-	<gazebo reference="realsense_link">
-    <gravity>true</gravity>
-    <sensor name="imu_realsense" type="imu">
-      <always_on>true</always_on>
-      <update_rate>20</update_rate>
-      <visualize>false</visualize>
-      <plugin name="imu_plugin" filename="libgazebo_ros_imu_sensor.so">
-        <topicName>imu_realsense/data_raw</topicName>
-        <bodyName>realsense_link</bodyName>
-        <updateRateHZ>100.0</updateRateHZ>
-        <gaussianNoise>0.0</gaussianNoise>
-        <xyzOffset>0 0 0</xyzOffset>
-        <rpyOffset>${-20*pi/180} 0 0</rpyOffset>
-        <frameName>realsense_link</frameName>
-        <initialOrientationAsReference>false</initialOrientationAsReference>
-      </plugin>
-    </sensor>
-  </gazebo>
+    <xacro:macro name="wheel_gazebo" params="prefix">
+        <gazebo reference="${prefix}_wheel_link">
+            <material>Gazebo/Grey</material>
+            <mu1>1</mu1>
+            <mu2>1</mu2>
+        </gazebo>
+    </xacro:macro>
+    <gazebo reference="base_link">
+        <material>Gazebo/Blue</material>
+    </gazebo>
+    <gazebo reference="realsense_link">
+        <sensor name="realsense_camera" type="depth">
+            <update_rate>10</update_rate>
+            <camera>
+                <pose>0 0 0 ${pi/2} ${-pi/2} 0</pose>
+                <horizontal_fov>1.5708</horizontal_fov>
+                <image>
+                    <width>640</width>
+                    <height>480</height>
+                    <format>R8G8B8</format>
+                </image>
+                <clip>
+                    <near>0.2</near>
+                    <far>4.0</far>
+                </clip>
+            </camera>
+            <plugin name="depth_camera_plugin" filename="libgazebo_ros_openni_kinect.so">
+                <alwaysOn>true</alwaysOn>
+                <updateRate>0.0</updateRate>
+                <cameraName>realsense</cameraName>
+                <frameName>realsense_link</frameName>
+                <imageTopicName>color/image_raw</imageTopicName>
+                <cameraInfoTopicName>color/camera_info</cameraInfoTopicName>
+                <depthImageTopicName>depth/image_raw</depthImageTopicName>
+                <depthImageInfoTopicName>depth/camera_info</depthImageInfoTopicName>
+                <pointCloudTopicName>depth/points</pointCloudTopicName>
+                <pointCloudCutoff>0.2</pointCloudCutoff>
+                <pointCloudCutoffMax>4.0</pointCloudCutoffMax>
+                <distortionK1>0.0</distortionK1>
+                <distortionK2>0.0</distortionK2>
+                <distortionK3>0.0</distortionK3>
+                <distortionT1>0.0</distortionT1>
+                <distortionT2>0.0</distortionT2>
+                <CxPrime>0</CxPrime>
+                <Cx>0</Cx>
+                <Cy>0</Cy>
+                <focalLength>0</focalLength>
+            </plugin>
+        </sensor>
+    </gazebo>
+    <!-- gazebo_ros_p3d for position groundtruth -->
+    <gazebo>
+        <plugin name="p3d_base_link_controller" filename="libcustom_p3d_plugin.so">
+            <alwaysOn>true</alwaysOn>
+            <updateRate>5.0</updateRate>
+            <bodyName>base_link</bodyName>
+            <topicName>/uwb_nodes</topicName>
+            <frameName>map</frameName>
+            <xyzOffsets>0 0 0</xyzOffsets>
+            <rpyOffsets>0 0 0</rpyOffsets>
+            <gaussianNoise>0.15</gaussianNoise>
+        </plugin>
+    </gazebo>
+    <gazebo reference="realsense_link">
+        <gravity>true</gravity>
+        <sensor name="imu_realsense" type="imu">
+        <always_on>true</always_on>
+        <update_rate>20</update_rate>
+        <visualize>false</visualize>
+            <plugin name="imu_plugin" filename="libgazebo_ros_imu_sensor.so">
+                <topicName>imu_realsense/data_raw</topicName>
+                <bodyName>realsense_link</bodyName>
+                <updateRateHZ>100.0</updateRateHZ>
+                <gaussianNoise>0.01</gaussianNoise>
+                <xyzOffset>0 0 0</xyzOffset>
+                <rpyOffset>${-20*pi/180} 0 0</rpyOffset>
+                <frameName>realsense_link</frameName>
+                <initialOrientationAsReference>false</initialOrientationAsReference>
+            </plugin>
+        </sensor>
+    </gazebo>
+    <gazebo reference="imu_link">
+        <gravity>true</gravity>
+        <sensor name="imu_sensor" type="imu">
+        <always_on>true</always_on>
+        <update_rate>30</update_rate>
+        <visualize>false</visualize>
+        <topic>imu</topic>
+            <plugin filename="libgazebo_ros_imu_sensor.so" name="imu_plugin">
+                <topicName>imu</topicName>
+                <bodyName>imu_link</bodyName>
+                <updateRateHZ>30.0</updateRateHZ>
+                <gaussianNoise>0.01</gaussianNoise>
+                <xyzOffset>0 0 0</xyzOffset>
+                <rpyOffset>0 0 0</rpyOffset>
+                <frameName>imu_link</frameName>
+                <initialOrientationAsReference>false</initialOrientationAsReference>
+            </plugin>
+        <pose>0 0 0 0 0 0</pose>
+        </sensor>
+    </gazebo>
   <!-- Gazebo plugin for ROS Control -->
   <gazebo>
     <plugin name="gazebo_ros_control" filename="libgazebo_ros_control.so">
-			<legacyModeNS>true</legacyModeNS>
+            <legacyModeNS>true</legacyModeNS>
       <robotNamespace>/</robotNamespace>
     </plugin>

File: glennobi_description/urdf/glennobi.transmission.xacro (robot description, xacro)
@@ -1,6 +1,6 @@
 <?xml version="1.0"?>
 <robot name="glennobi_transmission_description" xmlns:xacro="http://www.ros.org/wiki/xacro">
-	<xacro:macro name="wheel_transmission" params="prefix">
-		<transmission name="${prefix}_wheel_trans">
+  <xacro:macro name="wheel_transmission" params="prefix">
+    <transmission name="${prefix}_wheel_trans">
       <type>transmission_interface/SimpleTransmission</type>
       <actuator name="${prefix}_wheel_motor">
@@ -11,4 +11,4 @@
       </joint>
     </transmission>
-	</xacro:macro>
+  </xacro:macro>
 </robot>

File: glennobi_description/urdf/glennobi.urdf.xacro (robot description, xacro)
@@ -1,89 +1,95 @@
 <?xml version="1.0"?>
 <robot name="glennobi" xmlns:xacro="http://www.ros.org/wiki/xacro">
-	<xacro:include filename="$(find glennobi_description)/urdf/glennobi.gazebo.xacro"/>
-	<xacro:include filename="$(find glennobi_description)/urdf/glennobi.transmission.xacro"/>
-	<xacro:property name="bodylength" value="1.3"/>
-	<xacro:property name="bodywidth" value="0.43"/>
-	<xacro:property name="bodyheight" value="0.35"/>
-	<xacro:property name="wheelradius" value="0.232"/>
-	<xacro:property name="wheelwidth" value="0.12"/>
-	<xacro:property name="wheelsepx" value="0.28"/>
-	<xacro:property name="wheelsepy" value="0.4"/>
-	<xacro:property name="wheeloffsetx" value="0.13"/>
-	<xacro:property name="bodyx" value="0.51"/>
-	<xacro:property name="bodyz" value="-0.05"/>
-	 <xacro:macro name="default_inertial" params="mass">
-    <inertial>
-      <mass value="${mass}"/>
-      <inertia ixx="1.0" ixy="0.0" ixz="0.0" iyy="1.0" iyz="0.0" izz="1.0" />
-    </inertial>
-  </xacro:macro>
-	<xacro:macro name="wheel" params="prefix side reflect">
-		<link name="${prefix}_wheel_link">
-			<visual>
-				<origin xyz="0 0 0" rpy="${pi/2} 0 0"/>
-				<geometry>
-					<cylinder radius="${wheelradius}" length="${wheelwidth}"/>
-				</geometry>
-			</visual>
-			<collision>
-				<!-- cylinder origin different than mesh origin -->
-				<origin xyz="0 0 0" rpy="${pi/2} 0 0"/>
-				<geometry>
-					<cylinder radius="${wheelradius}" length="${wheelwidth}"/>
-				</geometry>
-			</collision>
-			<inertial>
-				<mass value="1.6"/>
-				<inertia ixx="0.035" ixy="0.0" ixz="0.0" iyy="0.035" iyz="0.0" izz="0.06" />
-			</inertial>
-		</link>
-		<!-- set gazebo wheel properties -->
-		<xacro:wheel_gazebo prefix="${prefix}"/>
-		<joint name="${prefix}_wheel_joint" type="continuous">
-			<parent link="base_link"/>
-			<child link="${prefix}_wheel_link"/>
-			<origin xyz="${side*wheelsepx + wheeloffsetx} ${reflect*(wheelsepy/2 + wheelwidth/2)} 0"/>
-			<axis xyz="0 1 0"/>
-			<dynamics damping="0.8" friction="2.0"/>
-		</joint>
-		<!-- set wheel transmission properties -->
-		<xacro:wheel_transmission prefix="${prefix}"/>
-	</xacro:macro>
-	<link name="base_link">
-		<visual>
-			<origin xyz="${bodyx} 0 ${bodyz}" rpy="${pi/2} 0 ${pi/2}"/>
-			<geometry>
-					<mesh filename="package://glennobi_description/meshes/chassis.dae"/>
-			</geometry>
-		</visual>
-		<collision>
-			<origin xyz="${bodyx} 0 ${bodyz}" rpy="${pi/2} 0 ${pi/2}"/>
-			<geometry>
-				<mesh filename="package://glennobi_description/meshes/chassis.dae"/>
-				<!-- box size="${bodylength} ${bodywidth} ${bodyheight}"/-->
-			</geometry>
-		</collision>
-		<inertial>
-			<mass value="16"/>
-			<inertia ixx="4.5" ixy="0.0" ixz="0.0" iyy="4.5" iyz="0.0" izz="0.8" />
-		</inertial>
-	</link>
-	<xacro:wheel prefix="front_right" side="1" reflect="-1"/>
-	<xacro:wheel prefix="front_left" side="1" reflect="1"/>
-	<xacro:wheel prefix="back_right" side="-1" reflect="-1"/>
-	<xacro:wheel prefix="back_left" side="-1" reflect="1"/>
-	<link name="realsense_link">
-		<visual>
-			<geometry>
-				<box size="0.1 0.025 0.015"/>
-			</geometry>
-		</visual>
-	</link>
-	<joint name="realsense_joint" type="fixed">
-		<parent link="base_link"/>
-		<child link="realsense_link"/>
-		<!-- transform from base_link with additional 20 degree tilt down -->
-		<origin xyz="-0.57 0 0.33" rpy="${-(20+90)*pi/180} 0 ${pi/2}"/>
-	</joint>
+    <xacro:include filename="$(find glennobi_description)/urdf/glennobi.gazebo.xacro"/>
+    <xacro:include filename="$(find glennobi_description)/urdf/glennobi.transmission.xacro"/>
+    <xacro:property name="bodylength" value="1.3"/>
+    <xacro:property name="bodywidth" value="0.43"/>
+    <xacro:property name="bodyheight" value="0.35"/>
+    <xacro:property name="wheelradius" value="0.232"/>
+    <xacro:property name="wheelwidth" value="0.12"/>
+    <xacro:property name="wheelsepx" value="0.28"/>
+    <xacro:property name="wheelsepy" value="0.4"/>
+    <xacro:property name="wheeloffsetx" value="0.13"/>
+    <xacro:property name="bodyx" value="0.51"/>
+    <xacro:property name="bodyz" value="-0.05"/>
+    <xacro:macro name="default_inertial" params="mass">
+        <inertial>
+          <mass value="${mass}"/>
+          <inertia ixx="1.0" ixy="0.0" ixz="0.0" iyy="1.0" iyz="0.0" izz="1.0" />
+        </inertial>
+    </xacro:macro>
+    <xacro:macro name="wheel" params="prefix side reflect">
+        <link name="${prefix}_wheel_link">
+            <visual>
+                <origin xyz="0 0 0" rpy="${pi/2} 0 0"/>
+                <geometry>
+                    <cylinder radius="${wheelradius}" length="${wheelwidth}"/>
+                </geometry>
+            </visual>
+            <collision>
+                <!-- cylinder origin different than mesh origin -->
+                <origin xyz="0 0 0" rpy="${pi/2} 0 0"/>
+                <geometry>
+                    <cylinder radius="${wheelradius}" length="${wheelwidth}"/>
+                </geometry>
+            </collision>
+            <inertial>
+                <mass value="1.6"/>
+                <inertia ixx="0.035" ixy="0.0" ixz="0.0" iyy="0.035" iyz="0.0" izz="0.06" />
+            </inertial>
+        </link>
+        <!-- set gazebo wheel properties -->
+        <xacro:wheel_gazebo prefix="${prefix}"/>
+        <joint name="${prefix}_wheel_joint" type="continuous">
+            <parent link="base_link"/>
+            <child link="${prefix}_wheel_link"/>
+            <origin xyz="${side*wheelsepx + wheeloffsetx} ${reflect*(wheelsepy/2 + wheelwidth/2)} 0"/>
+            <axis xyz="0 1 0"/>
+            <dynamics damping="0.8" friction="2.0"/>
+        </joint>
+        <!-- set wheel transmission properties -->
+        <xacro:wheel_transmission prefix="${prefix}"/>
+    </xacro:macro>
+    <link name="base_link">
+        <visual>
+            <origin xyz="${bodyx} 0 ${bodyz}" rpy="${pi/2} 0 ${pi/2}"/>
+            <geometry>
+                    <mesh filename="package://glennobi_description/meshes/chassis.dae"/>
+            </geometry>
+        </visual>
+        <collision>
+            <origin xyz="${bodyx} 0 ${bodyz}" rpy="${pi/2} 0 ${pi/2}"/>
+            <geometry>
+                <mesh filename="package://glennobi_description/meshes/chassis.dae"/>
+                <!-- box size="${bodylength} ${bodywidth} ${bodyheight}"/-->
+            </geometry>
+        </collision>
+        <inertial>
+            <mass value="16"/>
+            <inertia ixx="4.5" ixy="0.0" ixz="0.0" iyy="4.5" iyz="0.0" izz="0.8" />
+        </inertial>
+    </link>
+    <xacro:wheel prefix="front_right" side="1" reflect="-1"/>
+    <xacro:wheel prefix="front_left" side="1" reflect="1"/>
+    <xacro:wheel prefix="back_right" side="-1" reflect="-1"/>
+    <xacro:wheel prefix="back_left" side="-1" reflect="1"/>
+    <link name="realsense_link">
+        <visual>
+            <geometry>
+                <box size="0.1 0.025 0.015"/>
+            </geometry>
+        </visual>
+    </link>
+    <joint name="realsense_joint" type="fixed">
+        <parent link="base_link"/>
+        <child link="realsense_link"/>
+        <!-- transform from base_link with additional 20 degree tilt down -->
+        <origin xyz="-0.57 0 0.33" rpy="${-(20+90)*pi/180} 0 ${pi/2}"/>
+    </joint>
+    <link name="imu_link"/>
+    <joint name="imu_joint" type="fixed">
+        <parent link="base_link"/>
+        <child link="imu_link"/>
+        <origin xyz="0.35 -0.1 0" rpy="0 0 0"/>
+    </joint>
 </robot>
