Commit message: Small fixes (#23)
Make small improvements and basic state machine

File: glennobi_description/urdf/glennobi.gazebo.xacro (robot description, xacro)
@@ -1,91 +1,111 @@
 <?xml version="1.0"?>
 <robot name="glennobi_gazebo_description" xmlns:xacro="http://www.ros.org/wiki/xacro">
-	<xacro:macro name="wheel_gazebo" params="prefix">
-		<gazebo reference="${prefix}_wheel_link">
-			<material>Gazebo/Grey</material>
-			<mu1>3</mu1>
-			<mu2>3</mu2>
-		</gazebo>
-	</xacro:macro>
-	<gazebo reference="base_link">
-		<material>Gazebo/Blue</material>
-	</gazebo>
-	<gazebo reference="realsense_link">
-		<sensor name="realsense_camera" type="depth">
-			<update_rate>10</update_rate>
-			<camera>
-				<pose>0 0 0 ${pi/2} ${-pi/2} 0</pose>
-				<horizontal_fov>1.5708</horizontal_fov>
-				<image>
-					<width>640</width>
-					<height>480</height>
-					<format>R8G8B8</format>
-				</image>
-				<clip>
-					<near>0.2</near>
-					<far>4.0</far>
-				</clip>
-			</camera>
-			<plugin name="depth_camera_plugin" filename="libgazebo_ros_openni_kinect.so">
-				<alwaysOn>true</alwaysOn>
-				<updateRate>0.0</updateRate>
-				<cameraName>realsense</cameraName>
-				<frameName>realsense_link</frameName>
-				<imageTopicName>color/image_raw</imageTopicName>
-				<cameraInfoTopicName>color/camera_info</cameraInfoTopicName>
-				<depthImageTopicName>depth/image_raw</depthImageTopicName>
-				<depthImageInfoTopicName>depth/camera_info</depthImageInfoTopicName>
-				<pointCloudTopicName>depth/points</pointCloudTopicName>
-				<pointCloudCutoff>0.2</pointCloudCutoff>
-				<pointCloudCutoffMax>4.0</pointCloudCutoffMax>
-				<distortionK1>0.0</distortionK1>
-				<distortionK2>0.0</distortionK2>
-				<distortionK3>0.0</distortionK3>
-				<distortionT1>0.0</distortionT1>
-				<distortionT2>0.0</distortionT2>
-				<CxPrime>0</CxPrime>
-				<Cx>0</Cx>
-				<Cy>0</Cy>
-				<focalLength>0</focalLength>
-			</plugin>
-		</sensor>
-	</gazebo>
-	<!-- gazebo_ros_p3d for position groundtruth -->
-	<gazebo>
-		<plugin name="p3d_base_link_controller" filename="libcustom_p3d_plugin.so">
-				<alwaysOn>true</alwaysOn>
-				<updateRate>5.0</updateRate>
-				<bodyName>base_link</bodyName>
-				<topicName>/uwb_nodes</topicName>
-				<frameName>map</frameName>
-				<xyzOffsets>0 0 0</xyzOffsets>
-				<rpyOffsets>0 0 0</rpyOffsets>
-				<gaussianNoise>0.15</gaussianNoise>
-		</plugin>
-	</gazebo>
-	<gazebo reference="realsense_link">
-    <gravity>true</gravity>
-    <sensor name="imu_realsense" type="imu">
-      <always_on>true</always_on>
-      <update_rate>20</update_rate>
-      <visualize>false</visualize>
-      <plugin name="imu_plugin" filename="libgazebo_ros_imu_sensor.so">
-        <topicName>imu_realsense/data_raw</topicName>
-        <bodyName>realsense_link</bodyName>
-        <updateRateHZ>100.0</updateRateHZ>
-        <gaussianNoise>0.0</gaussianNoise>
-        <xyzOffset>0 0 0</xyzOffset>
-        <rpyOffset>${-20*pi/180} 0 0</rpyOffset>
-        <frameName>realsense_link</frameName>
-        <initialOrientationAsReference>false</initialOrientationAsReference>
-      </plugin>
-    </sensor>
-  </gazebo>
+    <xacro:macro name="wheel_gazebo" params="prefix">
+        <gazebo reference="${prefix}_wheel_link">
+            <material>Gazebo/Grey</material>
+            <mu1>1.5</mu1>
+            <mu2>1.5</mu2>
+        </gazebo>
+    </xacro:macro>
+    <gazebo reference="base_link">
+        <material>Gazebo/Blue</material>
+    </gazebo>
+    <gazebo reference="realsense_link">
+        <sensor name="realsense_camera" type="depth">
+            <update_rate>10</update_rate>
+            <camera>
+                <pose>0 0 0 ${pi/2} ${-pi/2} 0</pose>
+                <horizontal_fov>1.5708</horizontal_fov>
+                <image>
+                    <width>640</width>
+                    <height>480</height>
+                    <format>R8G8B8</format>
+                </image>
+                <clip>
+                    <near>0.2</near>
+                    <far>4.0</far>
+                </clip>
+            </camera>
+            <plugin name="depth_camera_plugin" filename="libgazebo_ros_openni_kinect.so">
+                <alwaysOn>true</alwaysOn>
+                <updateRate>0.0</updateRate>
+                <cameraName>realsense</cameraName>
+                <frameName>realsense_link</frameName>
+                <imageTopicName>color/image_raw</imageTopicName>
+                <cameraInfoTopicName>color/camera_info</cameraInfoTopicName>
+                <depthImageTopicName>depth/image_raw</depthImageTopicName>
+                <depthImageInfoTopicName>depth/camera_info</depthImageInfoTopicName>
+                <pointCloudTopicName>depth/points</pointCloudTopicName>
+                <pointCloudCutoff>0.2</pointCloudCutoff>
+                <pointCloudCutoffMax>4.0</pointCloudCutoffMax>
+                <distortionK1>0.0</distortionK1>
+                <distortionK2>0.0</distortionK2>
+                <distortionK3>0.0</distortionK3>
+                <distortionT1>0.0</distortionT1>
+                <distortionT2>0.0</distortionT2>
+                <CxPrime>0</CxPrime>
+                <Cx>0</Cx>
+                <Cy>0</Cy>
+                <focalLength>0</focalLength>
+            </plugin>
+        </sensor>
+    </gazebo>
+    <!-- gazebo_ros_p3d for position groundtruth -->
+    <gazebo>
+        <plugin name="p3d_base_link_controller" filename="libcustom_p3d_plugin.so">
+            <alwaysOn>true</alwaysOn>
+            <updateRate>5.0</updateRate>
+            <bodyName>base_link</bodyName>
+            <topicName>/uwb_nodes</topicName>
+            <frameName>map</frameName>
+            <xyzOffsets>0 0 0</xyzOffsets>
+            <rpyOffsets>0 0 0</rpyOffsets>
+            <gaussianNoise>0.15</gaussianNoise>
+        </plugin>
+    </gazebo>
+    <gazebo reference="realsense_link">
+        <gravity>true</gravity>
+        <sensor name="imu_realsense" type="imu">
+        <always_on>true</always_on>
+        <update_rate>20</update_rate>
+        <visualize>false</visualize>
+            <plugin name="imu_plugin" filename="libgazebo_ros_imu_sensor.so">
+                <topicName>imu_realsense/data_raw</topicName>
+                <bodyName>realsense_link</bodyName>
+                <updateRateHZ>100.0</updateRateHZ>
+                <gaussianNoise>0.01</gaussianNoise>
+                <xyzOffset>0 0 0</xyzOffset>
+                <rpyOffset>0 0 0</rpyOffset>
+                <frameName>realsense_link</frameName>
+                <initialOrientationAsReference>false</initialOrientationAsReference>
+            </plugin>
+        </sensor>
+    </gazebo>
+    <gazebo reference="imu_link">
+        <gravity>true</gravity>
+        <sensor name="imu_sensor" type="imu">
+        <always_on>true</always_on>
+        <update_rate>30</update_rate>
+        <visualize>false</visualize>
+        <topic>imu</topic>
+            <plugin filename="libgazebo_ros_imu_sensor.so" name="imu_plugin">
+                <topicName>imu</topicName>
+                <bodyName>imu_link</bodyName>
+                <updateRateHZ>30.0</updateRateHZ>
+                <gaussianNoise>0.01</gaussianNoise>
+                <xyzOffset>0 0 0</xyzOffset>
+                <rpyOffset>0 0 0</rpyOffset>
+                <frameName>imu_link</frameName>
+                <initialOrientationAsReference>false</initialOrientationAsReference>
+            </plugin>
+        <pose>0 0 0 0 0 0</pose>
+        </sensor>
+    </gazebo>
   <!-- Gazebo plugin for ROS Control -->
-  <gazebo>
-    <plugin name="gazebo_ros_control" filename="libgazebo_ros_control.so">
-			<legacyModeNS>true</legacyModeNS>
-      <robotNamespace>/</robotNamespace>
-    </plugin>
-  </gazebo>
+    <gazebo>
+        <plugin name="gazebo_ros_control" filename="libgazebo_ros_control.so">
+            <legacyModeNS>true</legacyModeNS>
+        <robotNamespace>/</robotNamespace>
+        </plugin>
+    </gazebo>
 </robot>

Commit message: In the middle of testing tf for realsense orientation

File: glennobi_description/urdf/glennobi.gazebo.xacro (robot description, xacro)
@@ -11,5 +11,5 @@
         <material>Gazebo/Blue</material>
     </gazebo>
-    <gazebo reference="realsense_link">
+    <gazebo reference="realsense_gyro_link">
         <sensor name="realsense_camera" type="depth">
             <update_rate>10</update_rate>
@@ -64,5 +64,5 @@
         </plugin>
     </gazebo>
-    <gazebo reference="realsense_link">
+    <gazebo reference="realsense_gyro_link">
         <gravity>true</gravity>
         <sensor name="imu_realsense" type="imu">
@@ -72,10 +72,10 @@
             <plugin name="imu_plugin" filename="libgazebo_ros_imu_sensor.so">
                 <topicName>imu_realsense/data_raw</topicName>
-                <bodyName>realsense_link</bodyName>
+                <bodyName>realsense_gyro_link</bodyName>
                 <updateRateHZ>100.0</updateRateHZ>
                 <gaussianNoise>0.01</gaussianNoise>
                 <xyzOffset>0 0 0</xyzOffset>
                 <rpyOffset>0 0 0</rpyOffset>
-                <frameName>realsense_link</frameName>
+                <frameName>realsense_gyro_link</frameName>
                 <initialOrientationAsReference>false</initialOrientationAsReference>
             </plugin>

File: glennobi_description/urdf/glennobi.urdf.xacro (robot description, xacro)
@@ -3,4 +3,5 @@
     <xacro:include filename="$(find glennobi_description)/urdf/glennobi.gazebo.xacro"/>
     <xacro:include filename="$(find glennobi_description)/urdf/glennobi.transmission.xacro"/>
+    <xacro:include filename="$(find glennobi_description)/urdf/realsense.urdf.xacro"/>
     <xacro:property name="bodylength" value="1.3"/>
     <xacro:property name="bodywidth" value="0.43"/>
@@ -74,17 +75,5 @@
     <xacro:wheel prefix="back_right" side="-1" reflect="-1"/>
     <xacro:wheel prefix="back_left" side="-1" reflect="1"/>
-    <link name="realsense_link">
-        <visual>
-            <geometry>
-                <box size="0.1 0.025 0.015"/>
-            </geometry>
-        </visual>
-    </link>
-    <joint name="realsense_joint" type="fixed">
-        <parent link="base_link"/>
-        <child link="realsense_link"/>
-        <!-- transform from base_link with additional 20 degree tilt down -->
-        <origin xyz="-0.57 0 0.33" rpy="${-(20+90)*pi/180} 0 ${pi/2}"/>
-    </joint>
+    <xacro:realsense name="realsense"/>
     <link name="imu_link"/>
     <joint name="imu_joint" type="fixed">

Commit message: Extremly minor tweaks

File: glennobi_description/urdf/glennobi.gazebo.xacro (robot description, xacro)
@@ -106,5 +106,5 @@
         <plugin name="gazebo_ros_control" filename="libgazebo_ros_control.so">
             <legacyModeNS>true</legacyModeNS>
-        <robotNamespace>/</robotNamespace>
+            <robotNamespace>/</robotNamespace>
         </plugin>
     </gazebo>

File: glennobi_description/urdf/glennobi.urdf.xacro (robot description, xacro)
@@ -64,14 +64,8 @@
     <xacro:property name="wheellxx" value="${1/12*wheelmass*(3*wheelradius*wheelradius+wheelwidth*wheelwidth)}"/>
     <xacro:property name="wheellxy" value="0.0"/>
-    <xacro:property name="wheellxz" value="0"/>
+    <xacro:property name="wheellxz" value="0.0"/>
     <xacro:property name="wheellyy" value="${1/2*wheelmass*wheelradius*wheelradius}"/>
     <xacro:property name="wheellyz" value="0.0"/>
     <xacro:property name="wheellzz" value="${wheellxx}"/>
-    <xacro:macro name="default_inertial" params="mass">
-        <inertial>
-          <mass value="${mass}"/>
-          <inertia ixx="1.0" ixy="0.0" ixz="0.0" iyy="1.0" iyz="0.0" izz="1.0" />
-        </inertial>
-    </xacro:macro>
     <xacro:macro name="wheel" params="prefix side reflect">
         <link name="${prefix}_wheel_link">
@@ -110,5 +104,5 @@
             <origin xyz="${bodyx} ${bodyy} ${bodyz}" rpy="${bodyroll} ${bodypitch} ${bodyyaw}"/>
             <geometry>
-                    <mesh filename="package://glennobi_description/meshes/chassis.dae"/>
+                <mesh filename="package://glennobi_description/meshes/chassis.dae"/>
             </geometry>
         </visual>

Commit message: New robot model2020 (#30)
* Refactor world and model files for simulator

* Added rock

* Create arena with holes world

* Add bumpy ground world and more

* Modify default world

* Fix a few camera transforms

* Reduce friction

File: glennobi_description/urdf/glennobi.gazebo.xacro (robot description, xacro)
@@ -4,6 +4,6 @@
         <gazebo reference="${prefix}_wheel_link">
             <material>Gazebo/Grey</material>
-            <mu1>1.5</mu1>
-            <mu2>1.5</mu2>
+            <mu1 value="0.6"/>
+            <mu2 value="0.6"/>
         </gazebo>
     </xacro:macro>
@@ -106,5 +106,5 @@
         <plugin name="gazebo_ros_control" filename="libgazebo_ros_control.so">
             <legacyModeNS>true</legacyModeNS>
-        <robotNamespace>/</robotNamespace>
+            <robotNamespace>/</robotNamespace>
         </plugin>
     </gazebo>

File: glennobi_description/urdf/glennobi.urdf.xacro (robot description, xacro)
@@ -3,19 +3,67 @@
     <xacro:include filename="$(find glennobi_description)/urdf/glennobi.gazebo.xacro"/>
     <xacro:include filename="$(find glennobi_description)/urdf/glennobi.transmission.xacro"/>
-    <xacro:property name="bodylength" value="1.3"/>
-    <xacro:property name="bodywidth" value="0.43"/>
-    <xacro:property name="bodyheight" value="0.35"/>
-    <xacro:property name="wheelradius" value="0.232"/>
-    <xacro:property name="wheelwidth" value="0.12"/>
-    <xacro:property name="wheelsepx" value="0.28"/>
-    <xacro:property name="wheelsepy" value="0.4"/>
-    <xacro:property name="wheeloffsetx" value="0.13"/>
-    <xacro:property name="bodyx" value="0.51"/>
-    <xacro:property name="bodyz" value="-0.05"/>
-    <xacro:macro name="default_inertial" params="mass">
-        <inertial>
-          <mass value="${mass}"/>
-          <inertia ixx="1.0" ixy="0.0" ixz="0.0" iyy="1.0" iyz="0.0" izz="1.0" />
-        </inertial>
+    <!-- NOTE Length=x, Width=y, Height=z-->
+    <!-- Values for the robot body-->
+    <!-- Units in Meters-->
+    <xacro:property name="bodylength" value="0.4577"/>
+    <xacro:property name="bodywidth" value="0.9411"/>
+    <xacro:property name="bodyheight" value="0.477"/>
+    <xacro:property name="wheelradius" value="0.1561"/>
+    <xacro:property name="wheelwidth" value="0.0762"/>
+    <!-- Distance from the centers of the wheels in the length and width of robot. -->
+    <!-- wheelsepx distance from spoke to spoke over 2 -->
+    <xacro:property name="wheelsepx" value="${0.3947/2}"/>
+    <!-- wheelsepy is from wheel to wheel not crossing the center line-->
+    <xacro:property name="wheelsepy" value="0.3175"/>
+    <!-- If wheels are not aligned use offset-->
+    <xacro:property name="wheeloffsetx" value="0.0"/>
+    <!-- body is for aligning the robot mesh to the center of gravity-->
+    <!-- Data from cad model
+    X = -2.54667
+	Y = 0.68615
+	Z = 9.90497
+    Note not currently used but leaving here because might be useful later-->
+    <xacro:property name="bodyx" value="0.13"/>
+    <xacro:property name="bodyy" value="0.01"/>
+    <xacro:property name="bodyz" value="0.12"/>
+    <!-- Controls tilt of robot model-->
+    <xacro:property name="bodyroll" value="0"/>
+    <xacro:property name="bodypitch" value="0"/>
+    <xacro:property name="bodyyaw" value="${pi/2}"/>
+    <!-- Note line up robot model first or you will spend time realigning the other sensors-->
+    <!-- Values for RealSense-->
+    <!-- Values for overall dimensions of RealSense-->
+    <xacro:property name="reallength" value="0.0758"/>
+    <xacro:property name="realwidth" value="0.025"/>
+    <xacro:property name="realheight" value="0.0151"/>
+    <!-- Values from center of Body to the RealSense-->
+    <xacro:property name="realx" value="${0.35+bodyx}"/>
+    <xacro:property name="realy" value="${0.152+bodyy}"/>
+    <xacro:property name="realz" value="${-0.01+bodyz}"/>
+    <!-- Controls tilt of RealSense model-->
+    <xacro:property name="realroll" value="${-(20.42 + 90) * pi/180}"/>
+    <xacro:property name="realpitch" value="0"/>
+    <xacro:property name="realyaw" value="${-pi/2}"/>
+    <!-- Inertia Section-->
+    <!-- Cadders Inertia Offset-->
+    <xacro:property name="robotlengthfromzero" value="-0.282549"/>
+    <xacro:property name="robotwidthfromzero" value="0.85221"/>
+    <xacro:property name="robotheightfromzero" value="-9.8254"/>
+    <!-- Masses unit kg-->
+    <xacro:property name="wheelmass" value="1.05216"/>
+    <!-- Mass of robot without wheels-->
+    <xacro:property name="robotmass" value="30.8"/>
+    <!-- Inertial values for robot units kg/m^2-->
+    <xacro:property name="robotlxx" value="0.385"/>
+    <xacro:property name="robotlxy" value="0"/>
+    <xacro:property name="robotlxz" value="0"/>
+    <xacro:property name="robotlyy" value="1.92098166"/>
+    <xacro:property name="robotlyz" value="0"/>
+    <xacro:property name="robotlzz" value="1.844169"/>
+    <!-- Inertial values for wheels units kg/m^2-->
+    <xacro:macro name="cylinder_inertia" params="m r h">
+      <inertia  ixx="${m*(3*r*r+h*h)/12}" ixy = "0" ixz = "0"
+        iyy="${m*(3*r*r+h*h)/12}" iyz = "0"
+        izz="${m*r*r/2}"/>
     </xacro:macro>
     <xacro:macro name="wheel" params="prefix side reflect">
@@ -35,6 +83,7 @@
             </collision>
             <inertial>
-                <mass value="1.6"/>
-                <inertia ixx="0.035" ixy="0.0" ixz="0.0" iyy="0.035" iyz="0.0" izz="0.06" />
+                <origin xyz="0 0 0" rpy="${pi/2} 0 0" />
+                <mass value="${wheelmass}"/>
+                <xacro:cylinder_inertia m="${wheelmass}" r="${wheelradius}" h="${wheelwidth}"/>
             </inertial>
         </link>
@@ -53,19 +102,19 @@
     <link name="base_link">
         <visual>
-            <origin xyz="${bodyx} 0 ${bodyz}" rpy="${pi/2} 0 ${pi/2}"/>
+            <origin xyz="${bodyx} ${bodyy} ${bodyz}" rpy="${bodyroll} ${bodypitch} ${bodyyaw}"/>
             <geometry>
-                    <mesh filename="package://glennobi_description/meshes/chassis.dae"/>
+                <mesh filename="package://glennobi_description/meshes/chassis.dae"/>
             </geometry>
         </visual>
         <collision>
-            <origin xyz="${bodyx} 0 ${bodyz}" rpy="${pi/2} 0 ${pi/2}"/>
+            <origin xyz="${bodyx} ${bodyy} ${bodyz}" rpy="${bodyroll} ${bodypitch} ${bodyyaw}"/>
             <geometry>
                 <mesh filename="package://glennobi_description/meshes/chassis.dae"/>
-                <!-- box size="${bodylength} ${bodywidth} ${bodyheight}"/-->
+                <!-- <box size="${bodylength} ${bodywidth} ${bodyheight}"/> -->
             </geometry>
         </collision>
         <inertial>
-            <mass value="16"/>
-            <inertia ixx="4.5" ixy="0.0" ixz="0.0" iyy="4.5" iyz="0.0" izz="0.8" />
+            <mass value="${robotmass}"/>
+            <inertia ixx="${robotlxx}" ixy="${robotlxy}" ixz="${robotlxz}" iyy="${robotlyy}" iyz="${robotlyz}" izz="${robotlzz}" />
         </inertial>
     </link>
@@ -77,5 +126,5 @@
         <visual>
             <geometry>
-                <box size="0.1 0.025 0.015"/>
+                <box size="${reallength} ${realwidth} ${realheight}"/>
             </geometry>
         </visual>
@@ -85,6 +134,7 @@
         <child link="realsense_link"/>
         <!-- transform from base_link with additional 20 degree tilt down -->
-        <origin xyz="-0.57 0 0.33" rpy="${-(20+90)*pi/180} 0 ${pi/2}"/>
+        <origin xyz="${realx} ${realy} ${realz}" rpy="${realroll} ${realpitch} ${realyaw}"/>
     </joint>
+    <!-- Waiting on this location from CAD people-->
     <link name="imu_link"/>
     <joint name="imu_joint" type="fixed">
