Commit message: Add imu_tools submodule and fix tf frames

File: glennobi_description/urdf/glennobi.gazebo.xacro (robot description, xacro)
@@ -11,12 +11,12 @@
         <material>Gazebo/Blue</material>
     </gazebo>
-    <gazebo reference="realsense_gyro_link">
+    <gazebo reference="realsense_link">
         <sensor name="realsense_camera" type="depth">
-            <update_rate>10</update_rate>
+            <update_rate>6</update_rate>
             <camera>
                 <pose>0 0 0 ${pi/2} ${-pi/2} 0</pose>
-                <horizontal_fov>1.5708</horizontal_fov>
+                <horizontal_fov>${radians(85.0)}</horizontal_fov>
                 <image>
-                    <width>640</width>
+                    <width>848</width>
                     <height>480</height>
                     <format>R8G8B8</format>
@@ -64,5 +64,5 @@
         </plugin>
     </gazebo>
-    <gazebo reference="realsense_gyro_link">
+    <gazebo reference="realsense_link">
         <gravity>true</gravity>
         <sensor name="imu_realsense" type="imu">
@@ -72,10 +72,10 @@
             <plugin name="imu_plugin" filename="libgazebo_ros_imu_sensor.so">
                 <topicName>imu_realsense/data_raw</topicName>
-                <bodyName>realsense_gyro_link</bodyName>
+                <bodyName>realsense_link</bodyName>
                 <updateRateHZ>100.0</updateRateHZ>
                 <gaussianNoise>0.01</gaussianNoise>
                 <xyzOffset>0 0 0</xyzOffset>
                 <rpyOffset>0 0 0</rpyOffset>
-                <frameName>realsense_gyro_link</frameName>
+                <frameName>realsense_link</frameName>
                 <initialOrientationAsReference>false</initialOrientationAsReference>
             </plugin>

File: glennobi_description/urdf/realsense.urdf.xacro (robot description, xacro)
@@ -21,9 +21,15 @@
     <!-- Our robot's coordinates to RealSense-->
     <xacro:macro name="realsense_origin">
-      <origin xyz="0.35 0.152 -0.01" rpy="${-(20.42 + 90) * pi/180} 0 ${-pi/2}"/>
+      <origin xyz="0.48 0.162 0.11" rpy="${-(20.42+90)*pi/180} 0 ${-pi/2}"/>
     </xacro:macro>
     <material name="${name}_aluminum">
       <color rgba="0.5 0.5 0.5 1"/>
     </material>
+    <link name="${name}_footprint_link"/>
+    <joint name="${name}_footprint_joint" type="fixed">
+      <parent link="base_link"/>
+      <child link="${name}_footprint_link"/>
+      <origin xyz="0.48 0.162 0.11" rpy="0 0 ${-pi/2}"/>
+    </joint>
     <link name="${name}_link">
       <visual>
@@ -43,15 +49,15 @@
     </link>
     <joint name="${name}_joint" type="fixed">
-      <parent link="base_link"/>
+      <parent link="${name}_footprint_link"/>
       <child link="${name}_link"/>
-      <xacro:realsense_origin/>
+      <origin xyz="0 0 0" rpy="${-radians(20.42 + 90)} 0 0"/>
     </joint>
-    <link name="${name}_gyro_link"/>
-    <joint name="${name}_gyro_joint" type="fixed">
-      <parent link="${name}_link"/>
-      <child link="${name}_gyro_link"/>
-      <!-- transform from realsense_link with additional 20 degree tilt down -->
-      <origin xyz="0 0 0" rpy="${-(20+90)*pi/180} 0 0"/>
-    </joint>
+    <!-- realsense_link will move due to imu data calulated with imu filter -->
+   <!--  <link name="${name}_link"/>
+    <joint name="${name}_joint" type="fixed">
+      <parent link="${name}_stabilized_link"/>
+      <child link="${name}_link"/>
+      <origin xyz="0 0 0" rpy="0 0 0"/>
+    </joint> -->
   </xacro:macro>
 </robot>

Commit message: Add tf for realsense orientation (#31)
* Use tf for global_occupancy_grid node

* Add imu_tools submodule and fix tf frames

* Integrate imu tilt detection

File: glennobi_description/urdf/glennobi.gazebo.xacro (robot description, xacro)
@@ -13,10 +13,10 @@
     <gazebo reference="realsense_link">
         <sensor name="realsense_camera" type="depth">
-            <update_rate>10</update_rate>
+            <update_rate>6</update_rate>
             <camera>
                 <pose>0 0 0 ${pi/2} ${-pi/2} 0</pose>
-                <horizontal_fov>1.5708</horizontal_fov>
+                <horizontal_fov>${radians(85.0)}</horizontal_fov>
                 <image>
-                    <width>640</width>
+                    <width>848</width>
                     <height>480</height>
                     <format>R8G8B8</format>
@@ -68,10 +68,10 @@
         <sensor name="imu_realsense" type="imu">
         <always_on>true</always_on>
-        <update_rate>20</update_rate>
+        <update_rate>40.0</update_rate>
         <visualize>false</visualize>
             <plugin name="imu_plugin" filename="libgazebo_ros_imu_sensor.so">
                 <topicName>imu_realsense/data_raw</topicName>
                 <bodyName>realsense_link</bodyName>
-                <updateRateHZ>100.0</updateRateHZ>
+                <updateRateHZ>40.0</updateRateHZ>
                 <gaussianNoise>0.01</gaussianNoise>
                 <xyzOffset>0 0 0</xyzOffset>

File: glennobi_description/urdf/glennobi.urdf.xacro (robot description, xacro)
@@ -3,4 +3,5 @@
     <xacro:include filename="$(find glennobi_description)/urdf/glennobi.gazebo.xacro"/>
     <xacro:include filename="$(find glennobi_description)/urdf/glennobi.transmission.xacro"/>
+    <xacro:include filename="$(find glennobi_description)/urdf/realsense.urdf.xacro"/>
     <!-- NOTE Length=x, Width=y, Height=z-->
     <!-- Values for the robot body-->
@@ -32,17 +33,4 @@
     <xacro:property name="bodyyaw" value="${pi/2}"/>
     <!-- Note line up robot model first or you will spend time realigning the other sensors-->
-    <!-- Values for RealSense-->
-    <!-- Values for overall dimensions of RealSense-->
-    <xacro:property name="reallength" value="0.0758"/>
-    <xacro:property name="realwidth" value="0.025"/>
-    <xacro:property name="realheight" value="0.0151"/>
-    <!-- Values from center of Body to the RealSense-->
-    <xacro:property name="realx" value="${0.35+bodyx}"/>
-    <xacro:property name="realy" value="${0.152+bodyy}"/>
-    <xacro:property name="realz" value="${-0.01+bodyz}"/>
-    <!-- Controls tilt of RealSense model-->
-    <xacro:property name="realroll" value="${-(20.42 + 90) * pi/180}"/>
-    <xacro:property name="realpitch" value="0"/>
-    <xacro:property name="realyaw" value="${-pi/2}"/>
     <!-- Inertia Section-->
     <!-- Cadders Inertia Offset-->
@@ -123,17 +111,5 @@
     <xacro:wheel prefix="back_right" side="-1" reflect="-1"/>
     <xacro:wheel prefix="back_left" side="-1" reflect="1"/>
-    <link name="realsense_link">
-        <visual>
-            <geometry>
-                <box size="${reallength} ${realwidth} ${realheight}"/>
-            </geometry>
-        </visual>
-    </link>
-    <joint name="realsense_joint" type="fixed">
-        <parent link="base_link"/>
-        <child link="realsense_link"/>
-        <!-- transform from base_link with additional 20 degree tilt down -->
-        <origin xyz="${realx} ${realy} ${realz}" rpy="${realroll} ${realpitch} ${realyaw}"/>
-    </joint>
+    <xacro:realsense name="realsense"/>
     <!-- Waiting on this location from CAD people-->
     <link name="imu_link"/>
