Commit message: renamed file names from glennobi to glenn

File: glenn_description/urdf/glenn.gazebo.xacro (robot description, xacro)
@@ -1,4 +1,4 @@
 <?xml version="1.0"?>
-<robot name="glennobi_gazebo_description" xmlns:xacro="http://www.ros.org/wiki/xacro">
+<robot name="glenn_gazebo_description" xmlns:xacro="http://www.ros.org/wiki/xacro">
     <xacro:macro name="wheel_gazebo" params="prefix">
         <gazebo reference="${prefix}_wheel_link">

File: glenn_description/urdf/glenn.transmission.xacro (robot description, xacro)
@@ -1,4 +1,4 @@
 <?xml version="1.0"?>
-<robot name="glennobi_transmission_description" xmlns:xacro="http://www.ros.org/wiki/xacro">
+<robot name="glenn_transmission_description" xmlns:xacro="http://www.ros.org/wiki/xacro">
   <xacro:macro name="wheel_transmission" params="prefix">
     <transmission name="${prefix}_wheel_trans">

File: glenn_description/urdf/glenn.urdf.xacro (robot description, xacro)
@@ -1,6 +1,6 @@
 <?xml version="1.0"?>
-<robot name="glennobi" xmlns:xacro="http://www.ros.org/wiki/xacro">
-    <xacro:include filename="$(find glennobi_description)/urdf/glennobi.gazebo.xacro"/>
-    <xacro:include filename="$(find glennobi_description)/urdf/glennobi.transmission.xacro"/>
+<robot name="glenn" xmlns:xacro="http://www.ros.org/wiki/xacro">
+    <xacro:include filename="$(find glenn_description)/urdf/glenn.gazebo.xacro"/>
+    <xacro:include filename="$(find glenn_description)/urdf/glenn.transmission.xacro"/>
     <!-- NOTE Length=x, Width=y, Height=z-->
     <!-- Values for the robot body-->
@@ -104,5 +104,5 @@
             <origin xyz="${bodyx} ${bodyy} ${bodyz}" rpy="${bodyroll} ${bodypitch} ${bodyyaw}"/>
             <geometry>
-                <mesh filename="package://glennobi_description/meshes/chassis.dae"/>
+                <mesh filename="package://glenn_description/meshes/chassis.dae"/>
             </geometry>
         </visual>
@@ -110,5 +110,5 @@
             <origin xyz="${bodyx} ${bodyy} ${bodyz}" rpy="${bodyroll} ${bodypitch} ${bodyyaw}"/>
             <geometry>
-                <mesh filename="package://glennobi_description/meshes/chassis.dae"/>
+                <mesh filename="package://glenn_description/meshes/chassis.dae"/>
                 <!-- <box size="${bodylength} ${bodywidth} ${bodyheight}"/> -->
             </geometry>

Commit message: Flat with rocks (#45)
* Added flat world with rocks

* renamed file names from glennobi to glenn

Co-authored-by: Ethan Frank <edf32@case.edu>

File: glenn_description/urdf/glenn.gazebo.xacro (robot description, xacro)
@@ -1,4 +1,4 @@
 <?xml version="1.0"?>
-<robot name="glennobi_gazebo_description" xmlns:xacro="http://www.ros.org/wiki/xacro">
+<robot name="glenn_gazebo_description" xmlns:xacro="http://www.ros.org/wiki/xacro">
     <xacro:macro name="wheel_gazebo" params="prefix">
         <gazebo reference="${prefix}_wheel_link">

File: glenn_description/urdf/glenn.urdf.xacro (robot description, xacro)
@@ -1,7 +1,7 @@
 <?xml version="1.0"?>
-<robot name="glennobi" xmlns:xacro="http://www.ros.org/wiki/xacro">
-    <xacro:include filename="$(find glennobi_description)/urdf/glennobi.gazebo.xacro"/>
-    <xacro:include filename="$(find glennobi_description)/urdf/glennobi.transmission.xacro"/>
-    <xacro:include filename="$(find glennobi_description)/urdf/realsense.urdf.xacro"/>
+<robot name="glenn" xmlns:xacro="http://www.ros.org/wiki/xacro">
+    <xacro:include filename="$(find glenn_description)/urdf/glenn.gazebo.xacro"/>
+    <xacro:include filename="$(find glenn_description)/urdf/glenn.transmission.xacro"/>
+    <xacro:include filename="$(find glenn_description)/urdf/realsense.urdf.xacro"/>
     <!-- NOTE Length=x, Width=y, Height=z-->
     <!-- Values for the robot body-->
@@ -92,5 +92,5 @@
             <origin xyz="${bodyx} ${bodyy} ${bodyz}" rpy="${bodyroll} ${bodypitch} ${bodyyaw}"/>
             <geometry>
-                <mesh filename="package://glennobi_description/meshes/chassis.dae"/>
+                <mesh filename="package://glenn_description/meshes/chassis.dae"/>
             </geometry>
         </visual>
@@ -98,5 +98,5 @@
             <origin xyz="${bodyx} ${bodyy} ${bodyz}" rpy="${bodyroll} ${bodypitch} ${bodyyaw}"/>
             <geometry>
-                <mesh filename="package://glennobi_description/meshes/chassis.dae"/>
+                <mesh filename="package://glenn_description/meshes/chassis.dae"/>
                 <!-- <box size="${bodylength} ${bodywidth} ${bodyheight}"/> -->
             </geometry>
