Commit message: added baselink

File: glenn_description/urdf/glenn.urdf.xacro (robot description, xacro)
@@ -107,4 +107,12 @@
         </inertial>
     </link>
+    <link name="base_link_footprint">
+		<origin xyz="${bodyx} ${bodyy} ${bodyz}" rpy="${bodyroll} ${bodypitch} ${bodyyaw}"/>
+    </link>
+    <joint name="base_link_joint" type="fixed">
+	<origin xyz="0 0 ${bodyz}" rpy="0 0 0" />
+	<parent link="base_link_footprint"/>
+	<child link="base_link" />
+    </joint>
     <xacro:wheel prefix="front_right" side="1" reflect="-1"/>
     <xacro:wheel prefix="front_left" side="1" reflect="1"/>

Commit message: base_link to base_link_footprint

File: glenn_description/urdf/glenn.urdf.xacro (robot description, xacro)
@@ -111,7 +111,7 @@
     </link>
     <joint name="base_link_joint" type="fixed">
-	<origin xyz="0 0 ${bodyz}" rpy="0 0 0" />
-	<parent link="base_link_footprint"/>
-	<child link="base_link" />
+        <origin xyz="0 0 ${wheelradius}" rpy="0 0 0" />
+        <parent link="base_link_footprint"/>
+        <child link="base_link" />
     </joint>
     <xacro:wheel prefix="front_right" side="1" reflect="-1"/>
