Commit message: Work on collision checking plugin

File: glenn_simulation/glenn_description/urdf/glenn.gazebo.xacro (robot description, xacro)
@@ -102,4 +102,15 @@
         </sensor>
     </gazebo>
+    <gazebo reference="base_link">
+        <sensor name="contact_sensor" type="contact">
+            <always_on>true</always_on>
+            <update_rate>5.0</update_rate>
+            <contact>
+                <collision>base_link_collision</collision>
+            </contact>
+            <plugin name="collisions_publisher" filename="libcollisions_publisher_plugin.so">
+            </plugin>
+        </sensor>
+    </gazebo>
   <!-- Gazebo plugin for ROS Control -->
     <gazebo>

Commit message: Modify files so they don't affect the rest of the code

File: glenn_simulation/glenn_description/urdf/glenn.gazebo.xacro (robot description, xacro)
@@ -102,15 +102,4 @@
         </sensor>
     </gazebo>
-    <gazebo reference="base_link">
-        <sensor name="contact_sensor" type="contact">
-            <always_on>true</always_on>
-            <update_rate>5.0</update_rate>
-            <contact>
-                <collision>base_link_collision</collision>
-            </contact>
-            <plugin name="collisions_publisher" filename="libcollisions_publisher_plugin.so">
-            </plugin>
-        </sensor>
-    </gazebo>
   <!-- Gazebo plugin for ROS Control -->
     <gazebo>
