Commit message: Reformat slighlty

File: glenn_simulation/glenn_description/urdf/glenn.urdf.xacro (robot description, xacro)
@@ -22,6 +22,6 @@
     <!-- Data from cad model
     X = -2.54667
-	Y = 0.68615
-	Z = 9.90497
+    Y = 0.68615
+    Z = 9.90497
     Note not currently used but leaving here because might be useful later-->
     <xacro:property name="bodyx" value="0.13"/>
@@ -107,7 +107,9 @@
         </inertial>
     </link>
+    <!-- Create a root link with no inertia to make the solver happy and raise the robot above the floor -->
     <link name="base_link_footprint">
-		<origin xyz="${bodyx} ${bodyy} ${bodyz}" rpy="${bodyroll} ${bodypitch} ${bodyyaw}"/>
+        <origin xyz="${bodyx} ${bodyy} ${bodyz}" rpy="${bodyroll} ${bodypitch} ${bodyyaw}"/>
     </link>
+    <!-- Connect that link to the base link in the middle of the robot -->
     <joint name="base_link_joint" type="fixed">
         <origin xyz="0 0 ${wheelradius}" rpy="0 0 0" />

Commit message: Base link footprint (#96)
* added baselink

* base_link to base_link_footprint

* Reformat slighlty

* Change frame names

* Remove ekf sample

* Revert comment

Co-authored-by: Erik Earl <erikjearl@gmail.com>

File: glenn_simulation/glenn_description/urdf/glenn.urdf.xacro (robot description, xacro)
@@ -22,6 +22,6 @@
     <!-- Data from cad model
     X = -2.54667
-	Y = 0.68615
-	Z = 9.90497
+    Y = 0.68615
+    Z = 9.90497
     Note not currently used but leaving here because might be useful later-->
     <xacro:property name="bodyx" value="0.13"/>
@@ -107,4 +107,14 @@
         </inertial>
     </link>
+    <!-- Create a root link with no inertia to make the solver happy and raise the robot above the floor -->
+    <link name="base_link_footprint">
+        <origin xyz="${bodyx} ${bodyy} ${bodyz}" rpy="${bodyroll} ${bodypitch} ${bodyyaw}"/>
+    </link>
+    <!-- Connect that link to the base link in the middle of the robot -->
+    <joint name="base_link_joint" type="fixed">
+        <origin xyz="0 0 ${wheelradius}" rpy="0 0 0" />
+        <parent link="base_link_footprint"/>
+        <child link="base_link" />
+    </joint>
     <xacro:wheel prefix="front_right" side="1" reflect="-1"/>
     <xacro:wheel prefix="front_left" side="1" reflect="1"/>

Commit message: Slightly understand things better I think.

File: glenn_simulation/glenn_description/urdf/glenn.urdf.xacro (robot description, xacro)
@@ -108,5 +108,5 @@
     </link>
     <!-- Create a root link with no inertia to make the solver happy and raise the robot above the floor -->
-    <link name="base_link_footprint">
+    <link name="base_footprint">
         <origin xyz="${bodyx} ${bodyy} ${bodyz}" rpy="${bodyroll} ${bodypitch} ${bodyyaw}"/>
     </link>
@@ -114,5 +114,5 @@
     <joint name="base_link_joint" type="fixed">
         <origin xyz="0 0 ${wheelradius}" rpy="0 0 0" />
-        <parent link="base_link_footprint"/>
+        <parent link="base_footprint"/>
         <child link="base_link" />
     </joint>
